File: JB_CNC_0.9.kicad_pcb (KiCad board)
At the start: 2 copper layers, 80 parts, among them CON1 POWER_IN, J1 Arduino_Nano_Header, P1 Z_CTRL, P10 X_LIMIT_1, P11 Y_LIMIT_1, P12 Z_LIMIT_1, P13 FLUIDO, P14 X_LIMIT_2, P15 Y_LIMIT_2, P16 Z_LIMIT_2, P17 SPINDLE_PWR, P18 SPINDLE_LED_ON, P19 SPINDLE_DIRECTION, P2 Z_LIMIT, P20 RESET/ABORT, P21 START/RESUME, P22 FEED_HOLD, P23 SAFETY_DOOR, P24 ASPIRADOR, P25 earth, P26 SPINDLE_LED_OFF, P3 Y_CTRL, P4 Y_LIMIT, P5 X_CTRL, P6 X_LIMIT, P7 USB_TO_ARDUINO, P8 F_INV, P9 USB_SHIELD_INPUT, Q1 BC546, Q2 BC546, Q3 BC546, Q4 BC546, Q5 BC546, U1 CA3140, U2 LM7805CT, U3 CA3140, U4 74LS86

Commit message: Desenho da placa em andamento
Routing:
- net (no net): track 0.00 -> 36.4 mm
Changed lines of the file:
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@@
     (links 172)
     (no_connects 81)
-    (area -128.705 -22.48 240.765001 182.9212)
+    (area -128.705 22.98346 274.083451 149.54)
     (thickness 1.6)
     (drawings 4)
-    (tracks 638)
+    (tracks 640)
     (zones 0)
     (modules 80)
@@
   (gr_line (start 240.665 132.715) (end 240.665 42.545) (angle 90) (layer F.Fab) (width 0.2))
   (gr_line (start 50.8 132.715) (end 240.665 132.715) (angle 90) (layer F.Fab) (width 0.2))
+  (segment (start 20.701 42.799) (end 30.48 42.799) (width 0.8) (layer F.Cu) (net 0))
+  (segment (start 30.48 42.799) (end 49.276 24.003) (width 0.8) (layer F.Cu) (net 0))
   (segment (start 159.258 67.945) (end 161.29 67.945) (width 1.4) (layer B.Cu) (net 2))
   (segment (start 166.497 62.738) (end 169.037 62.738) (width 1.4) (layer B.Cu) (net 2))

Commit message: primeiro commit colaborativo
Routing:
- net (no net): track 36.4 -> 0.00 mm
Changed lines of the file:
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@@
-(kicad_pcb (version 4) (host pcbnew 4.0.2+dfsg1-2~bpo8+1-stable)
+(kicad_pcb (version 4) (host pcbnew 4.0.2-stable)
   (general
     (links 172)
@@
     (thickness 1.6)
     (drawings 4)
-    (tracks 640)
+    (tracks 638)
     (zones 0)
     (modules 80)
@@
   (gr_line (start 240.665 132.715) (end 240.665 42.545) (angle 90) (layer F.Fab) (width 0.2))
   (gr_line (start 50.8 132.715) (end 240.665 132.715) (angle 90) (layer F.Fab) (width 0.2))
-  (segment (start 20.701 42.799) (end 30.48 42.799) (width 0.8) (layer F.Cu) (net 0))
-  (segment (start 30.48 42.799) (end 49.276 24.003) (width 0.8) (layer F.Cu) (net 0))
   (segment (start 159.258 67.945) (end 161.29 67.945) (width 1.4) (layer B.Cu) (net 2))
   (segment (start 166.497 62.738) (end 169.037 62.738) (width 1.4) (layer B.Cu) (net 2))

Commit message: Mudei o pad
Parts:
- moved P25 11.7 mm to (200.3, 92.1)
Changed lines of the file:
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@@
   )
   (module Socket_Strips:Socket_Strip_Straight_1x01 (layer F.Cu)
-    (at 205.994 102.235)
+    (at 200.279 92.075)
     (descr "Through hole socket strip")
     (tags "socket strip")

Commit message: Trilhas finalizadas
Parts:
- removed 1N1: 1N4001, Diodes_ThroughHole:Diode_DO-35_SOD27_Horizontal_RM10
- moved R5 287.8 mm to (178.4, 105.4), turned to 180 degrees
- moved R17 217.7 mm to (94.6, 117.5)
- moved R11 191.3 mm to (64.1, 122.6)
- moved R26 189.8 mm to (77.5, 126.4), turned to 180 degrees
- moved R25 181.7 mm to (98.6, 128.5)
- moved 1N4 178.7 mm to (77.5, 118.1)
- moved Q5 168.9 mm to (93.5, 128.5), turned to 180 degrees
- moved R27 161.3 mm to (64.1, 119.4)
- moved Q3 153.2 mm to (88.3, 123.8)
- moved R19 133.9 mm to (111.8, 116.8)
- moved 1N2 115.9 mm to (102.9, 124.5)
- moved Q2 83.3 mm to (188.0, 103.5)
- moved U3 83.2 mm to (181.9, 91.2)
- moved P8 83.2 mm to (170.8, 77.0)
- moved R15 83.2 mm to (185.6, 99.9)
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Connections:
- Q5 pad 2: GND -> Net-(P26-Pad2)
- Q5 pad 3: Net-(P26-Pad2) -> GND
- R25 pad 2: /SPINDLE_EN -> Net-(1N5-Pad2)
Routing:
- net +14V: track 51.6 -> 329.7 mm, vias 0 -> 6
- net GND: track 463.0 -> 702.8 mm, vias 7 -> 10
- net +5V: track 316.3 -> 442.9 mm, vias 6 -> 8
- net Net-(1N5-Pad2): track 0.00 -> 121.2 mm, vias 0 -> 2
- net /FEED_HOLD: track 4.21 -> 122.8 mm, vias 0 -> 2
- net /START/RESUME: track 24.5 -> 106.2 mm, vias 0 -> 2
- net /STEPPER_EN: track 86.2 -> 165.1 mm, vias 3 -> 6
- net /PROBE: track 0.00 -> 73.5 mm, vias 0 -> 2
- net /RESET/ABORT: track 17.0 -> 88.9 mm
- net /SPINDLE_DIR: track 0.00 -> 69.8 mm
- net /SPINDLE_PWM: track 15.9 -> 76.0 mm, vias 1 -> 2
- net Net-(P7-Pad3): track 0.00 -> 59.2 mm
- net /Z_LIMIT: track 0.00 -> 58.7 mm
- net Net-(P7-Pad2): track 0.00 -> 55.9 mm
- net /X_LIMIT: track 15.2 -> 68.0 mm, vias 0 -> 2
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
Commit message: Consertado erro de Esquema + Netlist
Parts:
- removed CON1: POWER_IN, Connect:BARREL_JACK
- added 1N1: 1N4001, Diodes_ThroughHole:Diode_DO-35_SOD27_Horizontal_RM10, F.Cu at (167.6, 120.4)
- added REF**: bornier2, Connect:bornier2, F.Cu at (158.5, 47.0)
- D2: footprint LEDs:LED-3MM -> LEDs:LED-5MM
- moved R1 10.0 mm to (167.1, 71.6), turned to 0 degrees
- moved Q5 5.77 mm to (87.8, 129.3), turned to 0 degrees
- moved D2 4.13 mm to (174.0, 46.2)
- moved C3 2.68 mm to (149.4, 46.1)
- moved P25 2.32 mm to (197.1, 105.8)
- moved R8 0.36 mm to (109.3, 91.4)
Connections:
- net /FEED_HOLD renamed /FEED_HOLD*
- net /RESET/ABORT renamed /RESET/ABORT*
- net /START/RESUME renamed /START/RESUME*
- net Net-(1N5-Pad2) renamed /SPINDLE_EN
- C1 pad 1: /SPINDLE_PWM -> Net-(C1-Pad1)
- C4 pad 1: /X_LIMIT_1 -> /X_LIMIT_A
- C5 pad 1: /Y_LIMIT_1 -> /Y_LIMIT_A
- C6 pad 1: /Z_LIMIT_1 -> /Z_LIMIT_A
- C7 pad 1: /X_LIMIT_2 -> /X_LIMIT_B
- C8 pad 1: /Y_LIMIT_2 -> /Y_LIMIT_B
- C9 pad 1: /Z_LIMIT_2 -> /Z_LIMIT_B
- P10 pad 3: /X_LIMIT_1 -> Net-(P10-Pad3)
- P11 pad 3: /Y_LIMIT_1 -> Net-(P11-Pad3)
- P12 pad 3: /Z_LIMIT_1 -> Net-(P12-Pad3)
- P14 pad 3: /X_LIMIT_2 -> Net-(P14-Pad3)
- P15 pad 3: /Y_LIMIT_2 -> Net-(P15-Pad3)
- P16 pad 3: /Z_LIMIT_2 -> Net-(P16-Pad3)
- P2 pad 1: /Z_LIMIT_1 -> /Z_LIMIT_A
- P2 pad 2: /Z_LIMIT_2 -> /Z_LIMIT_B
- P25 pad 1: Net-(P25-Pad1) -> GND
- P4 pad 1: /Y_LIMIT_1 -> /Y_LIMIT_A
- P4 pad 2: /Y_LIMIT_2 -> /Y_LIMIT_B
- P6 pad 1: /X_LIMIT_1 -> /X_LIMIT_A
- P6 pad 2: /X_LIMIT_2 -> /X_LIMIT_B
- P7 pad 5: Net-(P7-Pad5) -> (no net)
- P9 pad 5: Net-(P9-Pad5) -> (no net)
- Q5 pad 1: Net-(Q5-Pad1) -> Net-(P26-Pad2)
- Q5 pad 2: Net-(P26-Pad2) -> Net-(Q5-Pad2)
- R1 pad 2: /SPINDLE_PWM -> Net-(C1-Pad1)
- R10 pad 1: /Z_LIMIT_2 -> Net-(P16-Pad3)
- R10 pad 2: /Z_LIMIT_2 -> /Z_LIMIT_B
- R15 pad 2: /V_CTRL -> Net-(R15-Pad2)
- R25 pad 1: Net-(Q5-Pad1) -> Net-(Q5-Pad2)
- R3 pad 1: /X_LIMIT_1 -> Net-(P10-Pad3)
- R3 pad 2: /X_LIMIT_1 -> /X_LIMIT_A
- R6 pad 1: /Y_LIMIT_1 -> Net-(P11-Pad3)
- R6 pad 2: /Y_LIMIT_1 -> /Y_LIMIT_A
- R7 pad 1: /Z_LIMIT_1 -> Net-(P12-Pad3)
- R7 pad 2: /Z_LIMIT_1 -> /Z_LIMIT_A
- R8 pad 1: /X_LIMIT_2 -> Net-(P14-Pad3)
- R8 pad 2: /X_LIMIT_2 -> /X_LIMIT_B
- R9 pad 1: /Y_LIMIT_2 -> Net-(P15-Pad3)
- R9 pad 2: /Y_LIMIT_2 -> /Y_LIMIT_B
- U1 pad 3: /SPINDLE_PWM -> Net-(C1-Pad1)
- U3 pad 2: Net-(U3-Pad2) -> Net-(R15-Pad2)
- U3 pad 6: /V_CTRL -> Net-(R15-Pad2)
- U4 pad 1: /X_LIMIT_1 -> /X_LIMIT_A
- U4 pad 12: /Z_LIMIT_1 -> /Z_LIMIT_A
- U4 pad 13: /Z_LIMIT_2 -> /Z_LIMIT_B
- U4 pad 2: /X_LIMIT_2 -> /X_LIMIT_B
- U4 pad 4: /Y_LIMIT_1 -> /Y_LIMIT_A
- U4 pad 5: /Y_LIMIT_2 -> /Y_LIMIT_B
Routing:
- net /Z_LIMIT_B: track 0.00 -> 143.9 mm, vias 0 -> 2
- net /Z_LIMIT_2: track 139.0 -> 0.00 mm
- net /Z_LIMIT_1: track 106.8 -> 0.00 mm
- net /Y_LIMIT_2: track 103.3 -> 0.00 mm, vias 2 -> 0
- net /X_LIMIT_2: track 99.8 -> 0.00 mm, vias 3 -> 0
- net /Y_LIMIT_B: track 0.00 -> 97.4 mm, vias 0 -> 2
- net /Z_LIMIT_A: track 0.00 -> 86.2 mm
- net /Y_LIMIT_1: track 84.5 -> 0.00 mm
- net /X_LIMIT_B: track 0.00 -> 78.3 mm, vias 0 -> 2
- net /X_LIMIT_1: track 73.1 -> 0.00 mm, vias 4 -> 0
- net /Y_LIMIT_A: track 0.00 -> 66.8 mm
- net /X_LIMIT_A: track 0.00 -> 66.2 mm, vias 0 -> 4
- net GND: track 702.8 -> 750.8 mm, vias 10 -> 16
- net Net-(P12-Pad3): track 0.00 -> 20.6 mm
- net Net-(P14-Pad3): track 0.00 -> 19.6 mm, vias 0 -> 1
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
Commit message: Filtros Reprojetados
Parts:
- removed 1N5: 1N4001, Diodes_ThroughHole:Diode_DO-35_SOD27_Horizontal_RM10
- removed REF**: bornier2, Connect:bornier2
- added 1N3: 1N4001, Diodes_ThroughHole:Diode_DO-35_SOD27_Horizontal_RM10, F.Cu at (0.00, 0.00)
- added C13: 10u, Capacitors_ThroughHole:C_Radial_D5_L6_P2.5, F.Cu at (229.0, 30.0)
- added P27: SPINDLE_LED_OFF, w_conn_kk100:kk100_22-23-2021, F.Cu at (-1.27, 22.6)
- added R20: 10k, Resistors_ThroughHole:Resistor_Vertical_RM5mm, F.Cu at (-20.7, 20.1)
- added R22: 1k, Resistors_THT:Resistor_Vertical_RM5mm, F.Cu at (-7.49, -6.99)
- added R28: 2k7, Resistors_THT:Resistor_Vertical_RM5mm, F.Cu at (-4.57, 6.22)
- added R29: 1k, Resistors_THT:Resistor_Vertical_RM5mm, F.Cu at (4.70, -10.2)
- added R30: 10k, Resistors_ThroughHole:Resistor_Vertical_RM5mm, F.Cu at (-21.7, -4.32)
- added R31: 2k2, Resistors_ThroughHole:Resistor_Vertical_RM5mm, F.Cu at (0.00, 0.00)
- added R32: 10k, Resistors_ThroughHole:Resistor_Vertical_RM5mm, F.Cu at (0.00, 0.00)
- added W1: FONTE, Connect:bornier2, F.Cu at (-18.8, 3.81)
- C1: value 470nF -> 1uF
- C12: value 1uF -> 100u; footprint Capacitors_ThroughHole:C_Radial_D5_L6_P2.5 -> Capacitors_ThroughHole:C_Radial_D10_L13_P5
- C2: value 100u -> 1uF; footprint Capacitors_ThroughHole:C_Radial_D8_L11.5_P3.5 -> Capacitors_ThroughHole:C_Radial_D5_L6_P2.5
- C3: value 10u -> 1uF
- D2: footprint LEDs:LED-5MM -> LEDs:LED-3MM
- P13: value FLUIDO -> ASPIRADOR
- P18: value SPINDLE_LED_ON -> FLUIDO
- P19: value SPINDLE_DIRECTION -> RESETA/INTERROMPE
- P20: value RESET/ABORT -> INICIA/CONTINUA
- P21: value START/RESUME -> PAUSA
- P22: value FEED_HOLD -> SONDA
- P23: value SAFETY_DOOR -> PORTA_SEGURANÇA
- P24: value ASPIRADOR -> earth
- P25: value earth -> SPINDLE_LED_ON; footprint Socket_Strips:Socket_Strip_Straight_1x01 -> w_conn_kk100:kk100_22-23-2021
- P26: value SPINDLE_LED_OFF -> DIREÇÃO_SPINDLE
- P7: value USB_TO_ARDUINO -> USB_PARA_ARDUINO
- P9: value USB_SHIELD_INPUT -> ENTRADA_USB_SHIELD
- R1: value 100k -> 10k; footprint Resistors_ThroughHole:Resistor_Horizontal_RM10mm -> Resistors_ThroughHole:Resistor_Vertical_RM5mm
- R10, R12, R13, R21, R23, R3, R8, R9: value 22k -> 10k; footprint Resistors_ThroughHole:Resistor_Horizontal_RM10mm -> Resistors_ThroughHole:Resistor_Vertical_RM5mm
- R11, R17, R25, R26, R4, R5: footprint Resistors_ThroughHole:Resistor_Horizontal_RM10mm -> Resistors_ThroughHole:Resistor_Vertical_RM5mm
- R14: value 22k -> 2k7; footprint Resistors_ThroughHole:Resistor_Horizontal_RM10mm -> Resistors_ThroughHole:Resistor_Vertical_RM5mm
- R15: value 1k -> 680k; footprint Resistors_ThroughHole:Resistor_Horizontal_RM10mm -> Resistors_ThroughHole:Resistor_Vertical_RM5mm
- R16, R7: value 22k -> 68k; footprint Resistors_ThroughHole:Resistor_Horizontal_RM10mm -> Resistors_ThroughHole:Resistor_Vertical_RM5mm
- R18: value 6k2 -> 1k; footprint Resistors_ThroughHole:Resistor_Horizontal_RM10mm -> Resistors_ThroughHole:Resistor_Vertical_RM5mm
- R19: value 2k7 -> 1k; footprint Resistors_ThroughHole:Resistor_Horizontal_RM10mm -> Resistors_ThroughHole:Resistor_Vertical_RM5mm
- R2: value 6k2 -> 10k; footprint Resistors_ThroughHole:Resistor_Horizontal_RM10mm -> Resistors_ThroughHole:Resistor_Vertical_RM5mm
- R24: value 2k2 -> 1k; footprint Resistors_ThroughHole:Resistor_Horizontal_RM10mm -> Resistors_ThroughHole:Resistor_Vertical_RM5mm
- R27: value 10k -> 8k2; footprint Resistors_ThroughHole:Resistor_Horizontal_RM10mm -> Resistors_ThroughHole:Resistor_Vertical_RM5mm
- R6: value 22k -> 680k; footprint Resistors_ThroughHole:Resistor_Horizontal_RM10mm -> Resistors_ThroughHole:Resistor_Vertical_RM5mm
- U2: value LM7805CT -> CA3140; footprint TO_SOT_Packages_THT:TO-220_Neutral123_Horizontal_LargePads -> Housings_DIP:DIP-8_W7.62mm_LongPads
- U3: value CA3140 -> 7432; footprint Housings_DIP:DIP-8_W7.62mm_LongPads -> Housings_DIP:DIP-14_W7.62mm_LongPads
- U4: value 74LS86 -> LM7805CT; footprint Housings_DIP:DIP-14_W7.62mm_LongPads -> TO_SOT_Packages_THT:TO-220_Neutral123_Horizontal_LargePads
- moved 1N2 171.3 mm to (-64.6, 88.5)
- moved 1N4 171.3 mm to (-90.0, 82.1)
- moved C10 171.3 mm to (-95.9, 75.3)
- moved C11 171.3 mm to (-67.9, 75.0)
- moved P17 171.3 mm to (-50.0, 86.6)
- moved P18 171.3 mm to (-108.0, 83.8)
- moved P19 171.3 mm to (-84.3, 86.6)
- moved P20 171.3 mm to (-88.8, 74.5)
- moved P21 171.3 mm to (-88.8, 65.1)
- moved P22 171.3 mm to (-108.0, 65.0)
- moved P23 171.3 mm to (-108.0, 73.0)
- moved P24 171.3 mm to (-69.1, 86.6)
- moved P26 171.3 mm to (-108.0, 89.5)
- moved Q3 171.3 mm to (-79.2, 87.8)
- moved Q4 171.3 mm to (-55.1, 84.0)
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Connections:
- 1N1 pad 1: +14V -> VCC
- 1N2 pad 1: +14V -> VCC
- 1N2 pad 2: Net-(1N2-Pad2) -> /SPINDLE_EN
- 1N4 pad 1: +14V -> VCC
- C10 pad 1: /FEED_HOLD* -> /PROBE*
- C11 pad 1: /RESET/ABORT* -> /FEED_HOLD*
- C12 pad 1: /START/RESUME* -> VCC
- C2 pad 1: +14V -> /X_LIMIT_A
- C3 pad 1: +5V -> /Y_LIMIT_A
- C4 pad 1: /X_LIMIT_A -> /Z_LIMIT_A
- C5 pad 1: /Y_LIMIT_A -> /X_LIMIT_B
- C6 pad 1: /Z_LIMIT_A -> /Y_LIMIT_B
- C7 pad 1: /X_LIMIT_B -> /Z_LIMIT_B
- C8 pad 1: /Y_LIMIT_B -> /RESET/ABORT*
- C9 pad 1: /Z_LIMIT_B -> /START/RESUME*
- D1 pad 1: +14V -> VCC
- D2 pad 2: +14V -> VCC
- J1 pad 12: /X_LIMIT -> /X_LIMIT*
- J1 pad 13: /Y_LIMIT -> /Y_LIMIT*
- J1 pad 15: /Z_LIMIT -> /Z_LIMIT*
- J1 pad 24: /PROBE -> /PROBE*
- P13 pad 1: +14V -> VCC
- P17 pad 1: +14V -> VCC
- P18 pad 1: Net-(P18-Pad1) -> VCC
- P18 pad 2: GND -> Net-(1N3-Pad2)
- P19 pad 1: +14V -> +5V
- P19 pad 2: Net-(1N4-Pad2) -> Net-(P19-Pad2)
- P21 pad 2: Net-(P21-Pad2) -> /SAFETY_IN
- P22 pad 1: +5V -> GND
- P22 pad 2: /SAFETY_IN -> Net-(P22-Pad2)
- P24 pad 1: +14V -> GND
- P24 pad 2: Net-(1N2-Pad2) -> (no net)
- P25 pad 1: GND -> Net-(P25-Pad1)
- P26 pad 1: Net-(P26-Pad1) -> VCC
- P26 pad 2: Net-(P26-Pad2) -> Net-(1N4-Pad2)
- P7 pad 5: (no net) -> GND
- P9 pad 5: (no net) -> GND
- Q3 pad 1: Net-(1N4-Pad2) -> Net-(1N3-Pad2)
- Q4 pad 1: Net-(1N2-Pad2) -> Net-(1N4-Pad2)
- Q5 pad 1: Net-(P26-Pad2) -> Net-(P25-Pad2)
- R10 pad 1: Net-(P16-Pad3) -> Net-(P12-Pad3)
- R10 pad 2: /Z_LIMIT_B -> /Z_LIMIT_A
- R11 pad 1: Net-(P26-Pad1) -> Net-(P14-Pad3)
- R11 pad 2: +14V -> /X_LIMIT_B
- R12 pad 1: GND -> Net-(P15-Pad3)
- R12 pad 2: Net-(P20-Pad2) -> /Y_LIMIT_B
- R13 pad 1: GND -> Net-(P16-Pad3)
- R13 pad 2: Net-(P21-Pad2) -> /Z_LIMIT_B
- R14 pad 1: /START/RESUME* -> Net-(Q2-Pad2)
- R14 pad 2: Net-(P21-Pad2) -> /V_REF
- R15 pad 1: Net-(Q2-Pad2) -> VCC
- R15 pad 2: Net-(R15-Pad2) -> Net-(Q2-Pad2)
- R16 pad 1: GND -> VCC
- R16 pad 2: /SAFETY_IN -> Net-(Q2-Pad2)
- R17 pad 2: /SPINDLE_DIR -> /COOLANT_EN
- R18 pad 1: Net-(R18-Pad1) -> GND
- R18 pad 2: /V_CTRL -> Net-(P19-Pad2)
- R19 pad 1: Net-(Q4-Pad2) -> GND
- R19 pad 2: /PROBE -> Net-(P20-Pad2)
- R2 pad 2: Net-(R18-Pad1) -> Net-(R2-Pad2)
- R21 pad 1: /RESET/ABORT* -> /START/RESUME*
- R23 pad 1: /FEED_HOLD* -> /PROBE*
- R23 pad 2: Net-(P23-Pad3) -> Net-(P22-Pad2)
- R24 pad 1: Net-(D2-Pad1) -> GND
- R24 pad 2: GND -> /SAFETY_IN
- R25 pad 1: Net-(Q5-Pad2) -> /FEED_HOLD*
- R25 pad 2: /SPINDLE_EN -> Net-(P23-Pad3)
- R26 pad 1: +14V -> Net-(D2-Pad1)
- R26 pad 2: Net-(P26-Pad2) -> GND
- R27 pad 1: Net-(P18-Pad1) -> Net-(Q5-Pad2)
- R27 pad 2: Net-(P26-Pad2) -> /SPINDLE_EN
- R3 pad 1: Net-(P10-Pad3) -> Net-(R2-Pad2)
- R3 pad 2: /X_LIMIT_A -> /V_CTRL
- R5 pad 2: /COOLANT_EN -> /V_REF
- R6 pad 1: Net-(P11-Pad3) -> VCC
- R6 pad 2: /Y_LIMIT_A -> Net-(Q1-Pad2)
- R7 pad 1: Net-(P12-Pad3) -> VCC
- R7 pad 2: /Z_LIMIT_A -> Net-(Q1-Pad2)
- R8 pad 1: Net-(P14-Pad3) -> Net-(P10-Pad3)
- R8 pad 2: /X_LIMIT_B -> /X_LIMIT_A
- R9 pad 1: Net-(P15-Pad3) -> Net-(P11-Pad3)
- R9 pad 2: /Y_LIMIT_B -> /Y_LIMIT_A
- U1 pad 2: Net-(R18-Pad1) -> Net-(R2-Pad2)
- U1 pad 7: +14V -> VCC
- U2 pad 1: +14V -> Net-(U2-Pad1)
- U2 pad 2: GND -> /V_REF
- U2 pad 3: +5V -> /V_CTRL
- U3 pad 1: Net-(U3-Pad1) -> (no net)
- U3 pad 2: Net-(R15-Pad2) -> (no net)
- U3 pad 3: /V_CTRL -> (no net)
- U3 pad 4: GND -> /Z_LIMIT_B
- U3 pad 5: Net-(U3-Pad5) -> /Z_LIMIT_A
- U3 pad 6: Net-(R15-Pad2) -> /Z_LIMIT*
- U3 pad 7: +14V -> GND
- U3 pad 8: Net-(U3-Pad8) -> /Y_LIMIT*
- U4 pad 1: /X_LIMIT_A -> VCC
- U4 pad 2: /X_LIMIT_B -> GND
- U4 pad 3: /X_LIMIT -> +5V
Routing:
- net +14V: track 338.8 -> 0.00 mm, vias 6 -> 0
- net VCC: track 0.00 -> 260.1 mm, vias 0 -> 6
- net +5V: track 435.1 -> 200.4 mm, vias 8 -> 2
- net /STEPPER_EN: track 165.1 -> 22.8 mm, vias 6 -> 0
- net (no net): track 0.00 -> 127.5 mm
- net /FEED_HOLD*: track 122.8 -> 2.03 mm, vias 2 -> 0
- net /START/RESUME*: track 106.2 -> 4.29 mm, vias 2 -> 0
- net /RESET/ABORT*: track 88.9 -> 0.00 mm
- net /Z_LIMIT*: track 0.00 -> 77.5 mm
- net GND: track 750.8 -> 674.9 mm, vias 16 -> 17
- net /PROBE: track 73.5 -> 0.00 mm, vias 2 -> 0
- net /Y_LIMIT*: track 0.00 -> 71.0 mm
- net /SPINDLE_DIR: track 69.8 -> 0.00 mm
- net /X_LIMIT: track 68.0 -> 0.00 mm, vias 2 -> 0
- net /Z_DIR: track 147.5 -> 88.5 mm, vias 0 -> 1
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