File: JB_CNC_0.9.sch (KiCad schematic (older format))
At the start: 80 parts, among them CON1 POWER_IN, J1 Arduino_Nano_Header, P1 Z_CTRL, P10 X_LIMIT_1, P11 Y_LIMIT_1, P12 Z_LIMIT_1, P13 FLUIDO, P14 X_LIMIT_2, P15 Y_LIMIT_2, P16 Z_LIMIT_2, P17 SPINDLE_PWR, P18 SPINDLE_LED_ON, P19 SPINDLE_DIRECTION, P2 Z_LIMIT, P20 RESET/ABORT, P21 START/RESUME, P22 FEED_HOLD, P23 SAFETY_DOOR, P24 ASPIRADOR, P25 earth, P26 SPINDLE_LED_OFF, P3 Y_CTRL, P4 Y_LIMIT, P5 X_CTRL, P6 X_LIMIT, P7 USB_TO_ARDUINO, P8 F_INV, P9 USB_SHIELD_INPUT, Q1 BC546, Q2 BC546, Q3 BC546, Q4 BC546, Q5 BC546, U1 CA3140, U2 LM7805CT, U3 CA3140, U4 74LS86

Commit message: Consertado erro de Esquema + Netlist
Parts:
- CON1: footprint Connect:BARREL_JACK -> Connect:bornier2
- Q5: symbol BC817-40 -> BC546
Connections:
- net labels added: FEED_HOLD*, RESET/ABORT*, START/RESUME*, X_LIMIT_A, X_LIMIT_B, Y_LIMIT_A, Y_LIMIT_B, Z_LIMIT_A, Z_LIMIT_B
- net labels removed: Earth, FEED_HOLD, RESET/ABORT, START/RESUME, X_LIMIT_1, X_LIMIT_2, Y_LIMIT_1, Y_LIMIT_2, Z_LIMIT_1, Z_LIMIT_2
- wire segments 207 -> 208

Commit message: modificações acerca do probe
Parts:
- removed 1N2: 1N4001, Diodes_ThroughHole:Diode_DO-35_SOD27_Horizontal_RM10, symbol D
- removed Q4: BC546, TO_SOT_Packages_THT:TO-92_Inline_Wide, symbol BC546
- removed R19: 2k7, Resistors_ThroughHole:Resistor_Horizontal_RM10mm, symbol R
- added C?: 1uF, Capacitors_ThroughHole:C_Radial_D5_L6_P2.5, symbol C
- added R?: 22k, Resistors_ThroughHole:Resistor_Horizontal_RM10mm, symbol R
- P24: value ASPIRADOR -> PROBE
Connections:
- wire segments 208 -> 205
Other:
- note added: "Pino para entrada da sonda de contato\n(Referência variável para o eixo Z)\nPulldown com filtros para \ndebouncing (20ms).\n"
- note removed: "Pino para ativar e desativar o relé de alimentação\ndo aspirador\n\nDa mesma forma que foi feito na bomba de fluído \narrefecedor, deixa-se somente o pino para ativar e\ndesativar o relé de alimentação.\n"
Changed lines of the file:
@@
 L CONN_01X02 P24
 U 1 1 56AFBCA6
-P 15300 2650
-F 0 "P24" H 15300 2800 50  0001 C CNN
-F 1 "ASPIRADOR" V 15400 2650 50  0000 C CNN
-F 2 "w_conn_kk100:kk100_22-23-2021" H 15300 2650 50  0001 C CNN
-F 3 "" H 15300 2650 50  0000 C CNN
-	1    15300 2650
-	1    0    0    -1
-$EndComp
-Text Notes 13350 4100 0    60   ~ 0
-Pino para ativar e desativar o relé de alimentação\ndo aspirador\n\nDa mesma forma que foi feito na bomba de fluído \narrefecedor, deixa-se somente o pino  para ativar e\ndesativar o relé de alimentação.\n
+P 13600 2800
+F 0 "P24" H 13600 2950 50  0001 C CNN
+F 1 "PROBE" V 13700 2800 50  0000 C CNN
+F 2 "w_conn_kk100:kk100_22-23-2021" H 13600 2800 50  0001 C CNN
+F 3 "" H 13600 2800 50  0000 C CNN
+	1    13600 2800
+	-1   0    0    1
+$EndComp
 $Comp
 L CONN_01X02 P18
@@
 Text Notes 13700 6750 0    60   ~ 0
 Sinalizador de segurança SPINDLE_LED.\n\nQuando o spindle é ligado, o led_spindle_on \n(LED vermelho externo) é ativado, sinalizando\nque não é seguro mexer na máquina, pois o \nspindle está ligado, ou seja, a máquina está\nem operação. Quando o spindle é desligado,\nentão led_spindle_off (LED verde externo) é\nativado, sinalizando que é seguro mexer \nna máquina.
-Text Notes 10650 4550 0    60   ~ 0
+Text Notes 2250 -450 0    60   ~ 0
 Amplificação do sinal SPINDLE_DIR para\nutilizar no inversor de frequência:\n\nO relé de ativação das entradas do inversor\nde frequência é do tipo 12V, portanto usa-se\num circuito transistorizado para amplificar o\nsinal do arduíno de 5 para 14V com corrente\nsuficiente para ativar o relé.\n
 $Comp
@@
 L BC546 Q3
 U 1 1 57066D78
-P 11800 3350
-F 0 "Q3" H 12000 3425 50  0001 L CNN
-F 1 "BC546" H 11550 3150 50  0000 L CNN
-F 2 "TO_SOT_Packages_THT:TO-92_Inline_Wide" H 12000 3275 50  0001 L CIN
-F 3 "" H 11800 3350 50  0000 L CNN
-	1    11800 3350
+P 3250 -1650
+F 0 "Q3" H 3450 -1575 50  0001 L CNN
+F 1 "BC546" H 3000 -1850 50  0000 L CNN
+F 2 "TO_SOT_Packages_THT:TO-92_Inline_Wide" H 3450 -1725 50  0001 L CIN
+F 3 "" H 3250 -1650 50  0000 L CNN
+	1    3250 -1650
 	1    0    0    -1
 $EndComp
@@
 L R R17
 U 1 1 57066D7E
-P 11450 3350
-F 0 "R17" V 11525 3350 50  0001 C CNN
-F 1 "2k7" V 11450 3350 50  0000 C CNN
-F 2 "Resistors_ThroughHole:Resistor_Horizontal_RM10mm" V 11380 3350 50  0001 C CNN
-F 3 "" H 11450 3350 50  0000 C CNN
-	1    11450 3350
+P 2900 -1650
+F 0 "R17" V 2975 -1650 50  0001 C CNN
+F 1 "2k7" V 2900 -1650 50  0000 C CNN
+F 2 "Resistors_ThroughHole:Resistor_Horizontal_RM10mm" V 2830 -1650 50  0001 C CNN
+F 3 "" H 2900 -1650 50  0000 C CNN
+	1    2900 -1650
 	0    1    1    0
 $EndComp
@@
 L CONN_01X02 P19
 U 1 1 57066D8A
-P 12400 2900
-F 0 "P19" H 12400 3050 50  0001 C CNN
-F 1 "SPINDLE_DIRECTION" V 12550 2900 50  0000 C CNN
-F 2 "w_conn_kk100:kk100_22-23-2021" H 12400 2900 50  0001 C CNN
-F 3 "" H 12400 2900 50  0000 C CNN
-	1    12400 2900
+P 3850 -2100
+F 0 "P19" H 3850 -1950 50  0001 C CNN
+F 1 "SPINDLE_DIRECTION" V 4000 -2100 50  0000 C CNN
+F 2 "w_conn_kk100:kk100_22-23-2021" H 3850 -2100 50  0001 C CNN
+F 3 "" H 3850 -2100 50  0000 C CNN
+	1    3850 -2100
 	1    0    0    -1
 $EndComp
@@
 L GND-RESCUE-CapivaraCNC #PWR016
 U 1 1 57066D90
-P 11900 3600
-F 0 "#PWR016" H 11900 3600 30  0001 C CNN
-F 1 "GND" H 11900 3500 47  0000 C CNN
-F 2 "" H 11900 3600 60  0000 C CNN
-F 3 "" H 11900 3600 60  0000 C CNN
-	1    11900 3600
+P 3350 -1400
+F 0 "#PWR016" H 3350 -1400 30  0001 C CNN
+F 1 "GND" H 3350 -1500 47  0000 C CNN
+F 2 "" H 3350 -1400 60  0000 C CNN
+F 3 "" H 3350 -1400 60  0000 C CNN
+	1    3350 -1400
 	-1   0    0    -1
 $EndComp
@@
 L D 1N4
 U 1 1 57066DA3
-P 11900 2900
-F 0 "1N4" V 11875 3050 50  0001 C CNN
-F 1 "1N4001" H 11900 2800 50  0000 C CNN
-F 2 "Diodes_ThroughHole:Diode_DO-35_SOD27_Horizontal_RM10" H 11900 2900 50  0001 C CNN
-F 3 "" H 11900 2900 50  0000 C CNN
-	1    11900 2900
+P 3350 -2100
+F 0 "1N4" V 3325 -1950 50  0001 C CNN
+F 1 "1N4001" H 3350 -2200 50  0000 C CNN
+F 2 "Diodes_ThroughHole:Diode_DO-35_SOD27_Horizontal_RM10" H 3350 -2100 50  0001 C CNN
+F 3 "" H 3350 -2100 50  0000 C CNN
+	1    3350 -2100
 	0    1    1    0
 $EndComp
-Text Label 10700 3350 0    60   ~ 0
+Text Label 2150 -1650 0    60   ~ 0
 SPINDLE_DIR
-$Comp
-L BC546 Q4
-U 1 1 57067FB2
-P 14500 3100
-F 0 "Q4" H 14700 3175 50  0001 L CNN
-F 1 "BC546" H 14250 2900 50  0000 L CNN
-F 2 "TO_SOT_Packages_THT:TO-92_Inline_Wide" H 14700 3025 50  0001 L CIN
-F 3 "" H 14500 3100 50  0000 L CNN
-	1    14500 3100
-	1    0    0    -1
-$EndComp
-$Comp
-L R R19
-U 1 1 57067FB8
-P 14150 3100
-F 0 "R19" V 14225 3100 50  0001 C CNN
-F 1 "2k7" V 14150 3100 50  0000 C CNN
-F 2 "Resistors_ThroughHole:Resistor_Horizontal_RM10mm" V 14080 3100 50  0001 C CNN
-F 3 "" H 14150 3100 50  0000 C CNN
-	1    14150 3100
-	0    1    1    0
-$EndComp
-$Comp
-L GND #PWR017
-U 1 1 57067FCA
-P 14600 3300
-F 0 "#PWR017" H 14600 3300 30  0001 C CNN
-F 1 "GND" H 14600 3150 47  0000 C CNN
-F 2 "" H 14600 3300 60  0000 C CNN
-F 3 "" H 14600 3300 60  0000 C CNN
-	1    14600 3300
-	-1   0    0    -1
-$EndComp
-$Comp
-L D 1N2
-U 1 1 57067FDD
-P 14600 2650
-F 0 "1N2" V 14525 2775 50  0001 C CNN
-F 1 "1N4001" H 14600 2550 50  0000 C CNN
-F 2 "Diodes_ThroughHole:Diode_DO-35_SOD27_Horizontal_RM10" H 14600 2650 50  0001 C CNN
-F 3 "" H 14600 2650 50  0000 C CNN
-	1    14600 2650
-	0    1    1    0
-$EndComp
-Text Label 13600 3100 0    60   ~ 0
+Text Label 14450 2750 0    60   ~ 0
 PROBE
 $Comp
@@
 L +14V #PWR031
 U 1 1 58062D3D
-P 11900 2650
-F 0 "#PWR031" H 11900 2780 20  0001 C CNN
-F 1 "+14V" H 11905 2765 47  0000 C CNN
-F 2 "" H 11900 2650 60  0000 C CNN
-F 3 "" H 11900 2650 60  0000 C CNN
-	1    11900 2650
+P 3350 -2350
+F 0 "#PWR031" H 3350 -2220 20  0001 C CNN
+F 1 "+14V" H 3355 -2235 47  0000 C CNN
+F 2 "" H 3350 -2350 60  0000 C CNN
+F 3 "" H 3350 -2350 60  0000 C CNN
+	1    3350 -2350
 	1    0    0    -1
 $EndComp
@@
 F 3 "" H 14050 800 60  0000 C CNN
 	1    14050 800
-	1    0    0    -1
-$EndComp
-$Comp
-L +14V #PWR035
-U 1 1 5806548C
-P 14600 2400
-F 0 "#PWR035" H 14600 2530 20  0001 C CNN
-F 1 "+14V" H 14605 2515 47  0000 C CNN
-F 2 "" H 14600 2400 60  0000 C CNN
-F 3 "" H 14600 2400 60  0000 C CNN
-	1    14600 2400
 	1    0    0    -1
 $EndComp
@@
 Wire Notes Line
 	15950 4350 15950 6800
-Wire Notes Line
-	13050 2400 10550 2400
 Wire Wire Line
 	11600 5000 11600 6700
@@
 Wire Wire Line
 	9350 3400 9350 3550
-Connection ~ 11900 3100
-Wire Wire Line
-	11300 3350 10700 3350
-Wire Wire Line
-	14600 2400 14600 2500
-Wire Wire Line
-	14000 3100 13600 3100
+Connection ~ 3350 -1900
+Wire Wire Line
+	2750 -1650 2150 -1650
 Connection ~ 6350 4800
 Wire Wire Line
@@
 	15050 5350 15150 5350
 Wire Wire Line
-	11900 3100 12100 3100
-Wire Wire Line
-	11900 3050 11900 3150
+	3350 -1900 3550 -1900
+Wire Wire Line
+	3350 -1950 3350 -1850
 Wire Wire Line
 	6350 4750 6350 4850
@@
 Connection ~ 9200 3550
 Wire Wire Line
-	11900 2700 12100 2700
-Wire Wire Line
-	12100 2700 12100 2850
-Wire Wire Line
-	12100 2850 12200 2850
-Wire Wire Line
-	12200 2950 12100 2950
-Wire Wire Line
-	12100 2950 12100 3100
-Connection ~ 11900 2700
+	3350 -2300 3550 -2300
+Wire Wire Line
+	3550 -2300 3550 -2150
+Wire Wire Line
+	3550 -2150 3650 -2150
+Wire Wire Line
+	3650 -2050 3550 -2050
+Wire Wire Line
+	3550 -2050 3550 -1900
+Connection ~ 3350 -2300
 Wire Wire Line
 	3400 2200 4000 2200
@@
 	12850 600  15200 600
 Wire Wire Line
-	14600 2450 14900 2450
-Wire Wire Line
-	14900 2700 14900 2850
-Wire Wire Line
-	14900 2700 15100 2700
-Connection ~ 14600 2450
-Wire Wire Line
 	9350 3150 9350 3300
 Wire Wire Line
-	11900 2650 11900 2750
-Wire Wire Line
-	14900 2450 14900 2600
-Wire Wire Line
-	14900 2600 15100 2600
-Wire Wire Line
-	14600 2800 14600 2900
-Wire Wire Line
-	14900 2850 14600 2850
-Connection ~ 14600 2850
+	3350 -2350 3350 -2250
 Wire Wire Line
 	15000 5050 15050 5050
@@
 	13400 4350 15950 4350
 Wire Notes Line
-	13050 2400 13050 4600
-Wire Notes Line
-	10550 2400 10550 4600
+	4500 -2600 4500 -400
+Wire Notes Line
+	2000 -2600 2000 -400
 Wire Notes Line
 	6700 4050 4550 4050
-Wire Notes Line
-	15950 2200 13250 2200
 Wire Notes Line
 	4450 4000 1950 4000
@@
 	10850 600  10850 1950
 Wire Notes Line
-	10550 4600 13050 4600
+	2000 -400 4500 -400
 Wire Notes Line
 	10150 5900 7300 5900
@@
 Wire Notes Line
 	7200 6200 4850 6200
-Wire Notes Line
-	15950 2200 15950 4200
-Wire Notes Line
-	15950 4200 13250 4200
-Wire Notes Line
-	13250 4200 13250 2200
 Wire Wire Line
 	2950 2800 2900 2800
@@
 Wire Notes Line
 	10750 2450 6800 2450
+$Comp
+L R R?
+U 1 1 5849B1A5
+P 14100 2750
+F 0 "R?" V 14180 2750 50  0001 C CNN
+F 1 "22k" V 14100 2750 50  0000 C CNN
+F 2 "Resistors_ThroughHole:Resistor_Horizontal_RM10mm" V 14030 2750 50  0001 C CNN
+F 3 "" H 14100 2750 50  0000 C CNN
+	1    14100 2750
+	0    1    1    0
+$EndComp
+$Comp
+L C C?
+U 1 1 5849B1AB
+P 14300 2950
+F 0 "C?" H 14325 3050 50  0001 L CNN
+F 1 "1uF" H 14325 2850 50  0000 L CNN
+F 2 "Capacitors_ThroughHole:C_Radial_D5_L6_P2.5" H 14338 2800 50  0001 C CNN
+F 3 "" H 14300 2950 50  0000 C CNN
+	1    14300 2950
+	1    0    0    -1
+$EndComp
+$Comp
+L GND-RESCUE-CapivaraCNC #PWR?
+U 1 1 5849B1B1
+P 14300 3250
+F 0 "#PWR?" H 14300 3250 30  0001 C CNN
+F 1 "GND" H 14300 3150 47  0000 C CNN
+F 2 "" H 14300 3250 60  0000 C CNN
+F 3 "" H 14300 3250 60  0000 C CNN
+	1    14300 3250
+	-1   0    0    -1
+$EndComp
+Connection ~ 14300 2750
+Wire Wire Line
+	14300 2800 14300 2750
+Wire Wire Line
+	14250 2750 14750 2750
+Wire Wire Line
+	13950 2750 13800 2750
+Wire Wire Line
+	13800 2850 13800 3150
+Wire Wire Line
+	13800 3150 14300 3150
+Wire Wire Line
+	14300 3100 14300 3200
+Connection ~ 14300 3150
+Text Notes 13300 3800 0    60   ~ 0
+Pino para entrada da sonda de contato\n(Referência variável para o eixo Z)\nPulldown com filtros para \ndebouncing (20ms).\n
+Wire Notes Line
+	13250 2600 13250 3900
+Wire Notes Line
+	13250 3900 15200 3900
+Wire Notes Line
+	13250 2600 15200 2600
+Wire Notes Line
+	15200 2600 15200 3900
+Wire Notes Line
+	4500 -2600 2000 -2600
 $EndSCHEMATC

Commit message: Filtros Reprojetados
Parts:
- removed CON1: POWER_IN, Connect:bornier2, symbol BARREL_JACK
- removed R25: 10k, Resistors_ThroughHole:Resistor_Horizontal_RM10mm, symbol R
- removed U4: 74LS86, Housings_DIP:DIP-14_W7.62mm_LongPads, symbol 74LS86
- added 1N1: 1N4001, Diodes_ThroughHole:Diode_DO-35_SOD27_Horizontal_RM10, symbol D
- added P13: ASPIRADOR, w_conn_kk100:kk100_22-23-2021, symbol CONN_01X02
- added Q1: BC546, TO_SOT_Packages_THT:TO-92_Inline_Wide, symbol BC546
- added R15, R6: 680k, Resistors_ThroughHole:Resistor_Vertical_RM5mm, symbol R
- added R16, R7: 68k, Resistors_ThroughHole:Resistor_Vertical_RM5mm, symbol R
- added R22, R29: 1k, Resistors_ThroughHole:Resistor_Vertical_RM5mm, symbol R
- added R27: 8k2, Resistors_ThroughHole:Resistor_Vertical_RM5mm, symbol R
- added R5: 2k7, Resistors_ThroughHole:Resistor_Vertical_RM5mm, symbol R
- added U10: 74LS32, Housings_DIP:DIP-14_W7.62mm_LongPads, symbol 74LS32
- added W1: FONTE, Connect:bornier2, symbol BORNIER
- C1: value 470nF -> 1uF; footprint Capacitors_ThroughHole:C_Radial_D5_L6_P2.5 -> Capacitors_ThroughHole:C_Radial_D5_L11_P2.5
- C10: renamed from C?; footprint Capacitors_ThroughHole:C_Radial_D5_L6_P2.5 -> Capacitors_ThroughHole:C_Radial_D5_L11_P2.5; symbol C -> CP
- C11: renamed from C10; footprint Capacitors_ThroughHole:C_Radial_D5_L6_P2.5 -> Capacitors_ThroughHole:C_Radial_D5_L11_P2.5; symbol C -> CP
- C12: renamed from C2; footprint Capacitors_ThroughHole:C_Radial_D8_L11.5_P3.5 -> Capacitors_ThroughHole:C_Radial_D10_L13_P5
- C13: renamed from C3; footprint Capacitors_ThroughHole:C_Radial_D5_L6_P2.5 -> Capacitors_ThroughHole:C_Radial_D6.3_L11.2_P2.5
- C2: renamed from C4; footprint Capacitors_ThroughHole:C_Radial_D5_L6_P2.5 -> Capacitors_ThroughHole:C_Radial_D5_L11_P2.5; symbol C -> CP
- C3: renamed from C5; footprint Capacitors_ThroughHole:C_Radial_D5_L6_P2.5 -> Capacitors_ThroughHole:C_Radial_D5_L11_P2.5; symbol C -> CP
- C4: renamed from C6; footprint Capacitors_ThroughHole:C_Radial_D5_L6_P2.5 -> Capacitors_ThroughHole:C_Radial_D5_L11_P2.5; symbol C -> CP
- C5: renamed from C7; footprint Capacitors_ThroughHole:C_Radial_D5_L6_P2.5 -> Capacitors_ThroughHole:C_Radial_D5_L11_P2.5; symbol C -> CP
- C6: renamed from C8; footprint Capacitors_ThroughHole:C_Radial_D5_L6_P2.5 -> Capacitors_ThroughHole:C_Radial_D5_L11_P2.5; symbol C -> CP
- C7: renamed from C9; footprint Capacitors_ThroughHole:C_Radial_D5_L6_P2.5 -> Capacitors_ThroughHole:C_Radial_D5_L11_P2.5; symbol C -> CP
- C8: renamed from C11; footprint Capacitors_ThroughHole:C_Radial_D5_L6_P2.5 -> Capacitors_ThroughHole:C_Radial_D5_L11_P2.5; symbol C -> CP
- C9: renamed from C12; footprint Capacitors_ThroughHole:C_Radial_D5_L6_P2.5 -> Capacitors_ThroughHole:C_Radial_D5_L11_P2.5; symbol C -> CP
- D1: footprint Diodes_ThroughHole:Diode_DO-201AD_Horizontal_RM15 -> Diodes_ThroughHole:Diode_P600_Vertical_KathodeUp
- P19: renamed from P20; value RESET/ABORT -> RESETA/INTERROMPE
- P20: renamed from P21; value START/RESUME -> INICIA/CONTINUA
- P21: renamed from P22; value FEED_HOLD -> PAUSA
- P22: renamed from P24; value PROBE -> SONDA
- P23: value SAFETY_DOOR -> PORTA_SEGURANÇA
- P24: renamed from P25; footprint Socket_Strips:Socket_Strip_Straight_1x01 -> w_details:hole_1mm
- P25: renamed from P26; value SPINDLE_LED_OFF -> SPINDLE_LED_ON
- P26: renamed from P19; value SPINDLE_DIRECTION -> DIREÇÃO_SPINDLE
- P27: renamed from P18; value SPINDLE_LED_ON -> SPINDLE_LED_OFF
- P7: value USB_TO_ARDUINO -> USB_PARA_ARDUINO; footprint Connect:USB_A -> w_conn_pc:conn_usb_A; symbol USB_A -> USB_A-RESCUE-JB_CNC_0.9
- P9: value USB_SHIELD_INPUT -> ENTRADA_USB_SHIELD; footprint Connect:USB_B -> w_conn_pc:conn_usb_B; symbol USB_B -> USB_B-RESCUE-JB_CNC_0.9
- R1: value 100k -> 10k; footprint Resistors_ThroughHole:Resistor_Horizontal_RM10mm -> Resistors_ThroughHole:Resistor_Vertical_RM5mm
- R10: renamed from R7; value 22k -> 10k; footprint Resistors_ThroughHole:Resistor_Horizontal_RM10mm -> Resistors_ThroughHole:Resistor_Vertical_RM5mm
- R11: renamed from R8; value 22k -> 10k; footprint Resistors_ThroughHole:Resistor_Horizontal_RM10mm -> Resistors_ThroughHole:Resistor_Vertical_RM5mm
- R12: renamed from R9; value 22k -> 10k; footprint Resistors_ThroughHole:Resistor_Horizontal_RM10mm -> Resistors_ThroughHole:Resistor_Vertical_RM5mm
- R13: renamed from R10; value 22k -> 10k; footprint Resistors_ThroughHole:Resistor_Horizontal_RM10mm -> Resistors_ThroughHole:Resistor_Vertical_RM5mm
- R14: renamed from R15; value 1k -> 2k7; footprint Resistors_ThroughHole:Resistor_Horizontal_RM10mm -> Resistors_ThroughHole:Resistor_Vertical_RM5mm
- R17: renamed from R5; footprint Resistors_ThroughHole:Resistor_Horizontal_RM10mm -> Resistors_ThroughHole:Resistor_Vertical_RM5mm
- R18: renamed from R12; value 22k -> 1k; footprint Resistors_ThroughHole:Resistor_Horizontal_RM10mm -> Resistors_ThroughHole:Resistor_Vertical_RM5mm
- R19: renamed from R13; value 22k -> 1k; footprint Resistors_ThroughHole:Resistor_Horizontal_RM10mm -> Resistors_ThroughHole:Resistor_Vertical_RM5mm
- R2: value 6k2 -> 10k; footprint Resistors_ThroughHole:Resistor_Horizontal_RM10mm -> Resistors_ThroughHole:Resistor_Vertical_RM5mm
- R20: renamed from R21; value 22k -> 10k; footprint Resistors_ThroughHole:Resistor_Horizontal_RM10mm -> Resistors_ThroughHole:Resistor_Vertical_RM5mm
- R21: renamed from R14; value 22k -> 10k; footprint Resistors_ThroughHole:Resistor_Horizontal_RM10mm -> Resistors_ThroughHole:Resistor_Vertical_RM5mm
- R23: renamed from R?; value 22k -> 10k; footprint Resistors_ThroughHole:Resistor_Horizontal_RM10mm -> Resistors_ThroughHole:Resistor_Vertical_RM5mm
- R24: renamed from R16; value 22k -> 1k; footprint Resistors_ThroughHole:Resistor_Horizontal_RM10mm -> Resistors_ThroughHole:Resistor_Vertical_RM5mm
- R25: renamed from R23; value 22k -> 10k; footprint Resistors_ThroughHole:Resistor_Horizontal_RM10mm -> Resistors_ThroughHole:Resistor_Vertical_RM5mm
- R26: renamed from R24; footprint Resistors_ThroughHole:Resistor_Horizontal_RM10mm -> Resistors_ThroughHole:Resistor_Vertical_RM5mm
- R28: renamed from R17; footprint Resistors_ThroughHole:Resistor_Horizontal_RM10mm -> Resistors_ThroughHole:Resistor_Vertical_RM5mm
- R3: renamed from R18; value 6k2 -> 10k; footprint Resistors_ThroughHole:Resistor_Horizontal_RM10mm -> Resistors_ThroughHole:Resistor_Vertical_RM5mm
- R30: renamed from R11; footprint Resistors_ThroughHole:Resistor_Horizontal_RM10mm -> Resistors_ThroughHole:Resistor_Vertical_RM5mm
- R31: renamed from R26; footprint Resistors_ThroughHole:Resistor_Horizontal_RM10mm -> Resistors_ThroughHole:Resistor_Vertical_RM5mm
- R32: renamed from R27; footprint Resistors_ThroughHole:Resistor_Horizontal_RM10mm -> Resistors_ThroughHole:Resistor_Vertical_RM5mm
- R4: footprint Resistors_ThroughHole:Resistor_Horizontal_RM10mm -> Resistors_ThroughHole:Resistor_Vertical_RM5mm
- R8: renamed from R3; value 22k -> 10k; footprint Resistors_ThroughHole:Resistor_Horizontal_RM10mm -> Resistors_ThroughHole:Resistor_Vertical_RM5mm
- R9: renamed from R6; value 22k -> 10k; footprint Resistors_ThroughHole:Resistor_Horizontal_RM10mm -> Resistors_ThroughHole:Resistor_Vertical_RM5mm
- renumbered 1N5 to 1N2, 1N1 to 1N3, P13 to P18, Q1 to Q3, Q3 to Q4, U3 to U2, U2 to U4
Connections:
- net labels added: GNDPWR, PROBE*, VCC, V_REF, X_LIMIT*, Y_LIMIT*, Z_LIMIT*
- net labels removed: +14V, PROBE, X_LIMIT, Y_LIMIT, Z_LIMIT
- wire segments 205 -> 225
Other:
- note added: "Amplificação do sinal SPINDLE_DIR para\nutilizar no inversor de frequência:\n\nO relé de ativação das entradas do inversor\nde frequência é do tipo 12V, portanto usa-se\num circuito transistorizado para amplificar o\nsinal do arduíno de 5 para VCC com corrente\nsuficiente para ativar o relé.\n"
- note added: "Ativação do aspirador de acordo com spindle \n\nO aspirador deve sempre estar ligado enquanto\no spindle estiver em operação. Para isto, usa-se \num circuito transistorizado identico ao do spindle\nque ativa/desativa o relé do aspirador exatamente \nquando o relé de ativação do spindle for \nativado/desativado."
- note added: "Ativação/Desativação do spindle + aspirador via PWM:\n\nComo nessa versão do GRBL temos o pino SPINDLE_PWM\nsubstituindo o pino SPINDLE_EN, o spindle é ativado\ndiretamente no PWM do arduíno via GRBL. Como o valor V_CTRL\nnunca chega totalmente a zero, o spindle nunca pára.\nPara resolver esse problema, usa-se um circuito transistorizado\nque dá nível lógico zero na entrada de controle de ativaçã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"
- note added: "Circuito conversor Analog-Digital + Amplificador.\n\nComo o inversor de frequência utilizado trabalha \nsomente com valores analógicos de tensão, o sinal\ndo PWM é convertido para o valor equivalente de \ntensão analógica e amplificado para escala máxima\nde 0-10V de modo que o inversor de frequência \nreconheça o valor de velocidade que o GRBL solicita ."
- note added: "Fins de curso mecânicos. \nNormalmente fechados. Pulldown externo.\nPinos 1 e 2 podem ser NF ou NA,\ndependendo das lógica digital usada.\nDebounce: 15ms"
- note added: "Fonte: 15VDC VCC: 14.1 - 14.4V\nDiodo Ultra Rápido para Polarização Reversa.\nRegulador de Tensão para 5V."
- note added: "Logica digital de fim de curso:\nO arduíno detecta fim de curso\nsem diferenciar se o fim de curso\né máximo ou mínimo.\nOs drivers dos motores de passo \ndiferenciam isso, portanto sugere-se\nutilizar portas lógicas para isolar \no arduíno dos motores de passo\npara que ambos possam receber \ncomandos dos sensores de fim de \ncurso sem afetar um ao outro.\nObs.: Para lógica inversa\n(0 para HIGH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"
- note added: "Os botões de comando do GRBL usam\npullup interno por padrão, ou seja, \nATIVO-BAIXO com chave NA.\nUsam-se pulldown com filtros para \ndebouncing (15ms) e uma chave NF\npara manter o ACTIVE LOW.\n"
- note added: "Pino para entrada da sonda de contato\n(Referência variável para o eixo Z)\nPulldown com filtros para \ndebouncing (15ms).\n"
- note added: "Sensor da porta \nPino 1 NF\nPino 2 NA\nPino 3 Conn\nDebounce: 15ms\n"
- note added: "Sinalizador de segurança SPINDLE_LED.\n\nQuando o spindle é ligado, o LED_SPINDLE_ON \n(LED vermelho externo) é ativado, sinalizando\nque não é seguro mexer na máquina, pois o \nspindle está ligado, ou seja, a máquina está\nem operação. Quando o spindle é desligado,\nentão LED_SPINDLE_OFF (LED verde externo) é\nativado, sinalizando que é seguro mexer \nna máquina."
- note removed: "Amplificação do sinal SPINDLE_DIR para\nutilizar no inversor de frequência:\n\nO relé de ativação das entradas do inversor\nde frequência é do tipo 12V, portanto usa-se\num circuito transistorizado para amplificar o\nsinal do arduíno de 5 para 14V com corrente\nsuficiente para ativar o relé.\n"
- note removed: "Ativação e desativação do spindle via PWM:\n\nComo nessa versão do GRBL temos o pino\nSPINDLE_PWM substituindo o pino SPINDLE_EN,\no spindle é ativado diretamente no PWM do arduíno\nvia GRBL.\nComo o valor V_CTRL nunca chega totalmente a zero, \no spindle nunca pára.\nPara resolver esse problema, sugere-se um circuito\ntransistorizado que dá nível lógico zero na entrada de \ncontrole de ativação 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"
- note removed: "Circuito conversor Analog-Digital + Amplificador.\n\nComo o inversor de frequência utilizado trabalha \nsomente com valores analógicos de tensão, o sinal\ndo PWM é convertido para o valor equivalente de \ntensão analógica e amplificado numa escala máxima\nde 1:2.61 para trimmer setado no seu valor maximo (10k)\nde modo que o inversor de frequência reconheça\no valor de velocidade que o GRBL solic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"
- note removed: "Diodo Ultra Rápido para Polarização Reversa.\nRegulador de Tensão para 5V."
- note removed: "Fins de curso mecânicos. \nNormalmente fechados. Pulldown externo.\nPino 1 NF. Pino 2 NA. Pino 3 Conn.\nDebounce: 20ms"
- note removed: "Logica digital de fim de curso:\nO arduíno detecta fim de curso\nsem diferenciar se o fim de curso\né máximo ou mínimo.\nOs drivers dos motores de passo \ndiferenciam isso, portanto sugere-se\nutilizar portas lógicas para isolar \no arduíno dos motores de passo\npara que ambos possam receber \ncomandos dos sensores de fim de \ncurso sem afetar um ao outro.\nObs.: Para níveis lógicos invertidos\n(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"
- note removed: "Os botões de comando do GRBL usam\npullup interno por padrão, ou seja, \nACTIVE LOW com chave NA.\nUsarão-se pulldown com filtros para \ndebouncing (20ms) e uma chave NF\npara manter o ACTIVE LOW.\n"
- note removed: "Pino para entrada da sonda de contato\n(Referência variável para o eixo Z)\nPulldown com filtros para \ndebouncing (20ms).\n"
- note removed: "Sensor da porta \nPino 1 NF\nPino 2 NA\nPino 3 Conn\nDebounce: 20ms\n"
- note removed: "Sinalizador de segurança SPINDLE_LED.\n\nQuando o spindle é ligado, o led_spindle_on \n(LED vermelho externo) é ativado, sinalizando\nque não é seguro mexer na máquina, pois o \nspindle está ligado, ou seja, a máquina está\nem operação. Quando o spindle é desligado,\nentão led_spindle_off (LED verde externo) é\nativado, sinalizando que é seguro mexer \nna máquina."
- moved on the sheet: U1
