File: JB_CNC.kicad_pcb (KiCad board)
At the start: 2 copper layers, 94.5 x 155.5 mm, 96 parts, among them J1 Arduino_Nano_Header, P1 Z_CTRL, P10 X_LIMIT_1, P11 Y_LIMIT_1, P12 Z_LIMIT_1, P13 ASPIRADOR, P14 X_LIMIT_2, P15 Y_LIMIT_2, P16 Z_LIMIT_2, P17 SPINDLE_PWR, P18 FLUIDO, P19 RESETA/INTERROMPE, P2 Z_LIMIT, P20 INICIA/CONTINUA, P21 PAUSA, P22 SONDA, P23 PORTA_SEGURANÇA, P24 earth, P25 SPINDLE_LED_ON, P26 DIREÇÃO_SPINDLE, P27 SPINDLE_LED_OFF, P3 Y_CTRL, P4 Y_LIMIT, P5 X_CTRL, P6 X_LIMIT, P7 USB_PARA_ARDUINO, P8 F_INV, P9 ENTRADA_USB_SHIELD, Q1 BC546, Q2 BC546, Q3 BC546, Q4 BC546, Q5 BC546, U1 CA3140, U2 CA3140, U3 74LS86, U4 LM7805CT

Commit message: Finalizado Esquema V0.2
Parts:
- removed 1N2, 1N4: 1N4001, Diodes_ThroughHole:Diode_DO-35_SOD27_Horizontal_RM10
- removed AL1, AL2: Pin_Header_Angled_1x01, Pin_Headers:Pin_Header_Straight_1x01
- removed B0, B1, B2, B3, B4: Pin_Header_Straight_1x01, Pin_Headers:Pin_Header_Straight_1x01
- added D3: 1K5E68A, Diodes_ThroughHole:Diode_P600_Vertical_KathodeUp, F.Cu at (-26.5, 54.7)
- added R33: 1k, Resistors_ThroughHole:Resistor_Vertical_RM5mm, F.Cu at (43.5, 38.3)
- added R34: 1k, Resistors_ThroughHole:Resistor_Vertical_RM5mm, F.Cu at (12.9, 26.0)
- added R35: 4k7, Resistors_ThroughHole:Resistor_Vertical_RM5mm, F.Cu at (-11.3, -2.09)
- added R36: 1k, Resistors_ThroughHole:Resistor_Vertical_RM5mm, F.Cu at (4.70, -2.09)
- added R37: 4k7, Resistors_ThroughHole:Resistor_Vertical_RM5mm, F.Cu at (53.8, 62.3)
- added U10: 74LS32, Housings_DIP:DIP-14_W7.62mm_LongPads, F.Cu at (13.6, 145.4)
- added U5: 4N25, Housings_DIP:DIP-6_W7.62mm_LongPads, F.Cu at (30.0, 112.3)
- added U6: 4N25, Housings_DIP:DIP-6_W7.62mm_LongPads, F.Cu at (-11.4, 63.4)
- C1, C10, C11, C2, C3, C4, C5, C6, C7, C8, C9: footprint Capacitors_ThroughHole:C_Radial_D5_L6_P2.5 -> Capacitors_ThroughHole:C_Radial_D5_L11_P2.5
- C13: footprint Capacitors_ThroughHole:C_Radial_D5_L6_P2.5 -> Capacitors_ThroughHole:C_Radial_D6.3_L11.2_P2.5
- P17: footprint w_conn_kk100:kk100_22-23-2021 -> w_conn_kk100:kk100_22-23-2031
- P24: footprint w_details:pad_2mm -> w_details:hole_1mm
- P26: value DIREÇÃO_SPINDLE -> DIREÇÃO; footprint w_conn_kk100:kk100_22-23-2021 -> w_conn_kk100:kk100_22-23-2041
- P7: footprint Connect:USB_A -> w_conn_pc:conn_usb_A
- R1, R16, R17, R18, R19, R20, R21, R22, R23, R24, R25, R26, R4, R5, R7: footprint w_pth_resistors:RC03 -> Resistors_ThroughHole:Resistor_Vertical_RM5mm
- R10, R11, R12, R13, R8, R9: footprint w_pth_resistors:rc07_vert -> Resistors_ThroughHole:Resistor_Vertical_RM5mm
- R14: value 2k7 -> 10k; footprint w_pth_resistors:RC03 -> Resistors_ThroughHole:Resistor_Vertical_RM5mm
- R15: value 680k -> 470; footprint w_pth_resistors:RC03 -> Resistors_ThroughHole:Resistor_Vertical_RM5mm
- R2: value 10k -> 20k; footprint w_pth_resistors:RC03 -> Resistors_ThroughHole:Resistor_Vertical_RM5mm
- R27: value 8k2 -> 10k; footprint w_pth_resistors:rc07_vert -> Resistors_ThroughHole:Resistor_Vertical_RM5mm
- R28: value 2k7 -> 4k7; footprint w_pth_resistors:RC03 -> Resistors_ThroughHole:Resistor_Vertical_RM5mm
- R29: value 1k -> 10k; footprint w_pth_resistors:rc07_vert -> Resistors_ThroughHole:Resistor_Vertical_RM5mm
- R3: value 10k -> 22k; footprint w_pth_resistors:RC03 -> Resistors_ThroughHole:Resistor_Vertical_RM5mm
- R30, R32: value 10k -> 4k7; footprint w_pth_resistors:RC03 -> Resistors_ThroughHole:Resistor_Vertical_RM5mm
- R31: value 2k2 -> 1k; footprint w_pth_resistors:RC03 -> Resistors_ThroughHole:Resistor_Vertical_RM5mm
- R6: value 680k -> 1k; footprint w_pth_resistors:RC03 -> Resistors_ThroughHole:Resistor_Vertical_RM5mm
- U3: value 74LS86 -> 4N25; footprint Housings_DIP:DIP-14_W7.62mm_LongPads -> Housings_DIP:DIP-6_W7.62mm_LongPads
- U4: footprint TO_SOT_Packages_THT:TO-220_Neutral123_Horizontal_LargePads -> Power_Integrations:TO-220
- moved R1 228.8 mm to (12.7, -5.05)
- moved C4 212.4 mm to (-29.7, -4.43), turned to 90 degrees
- moved R3 203.4 mm to (4.30, -12.6), turned to 90 degrees
- moved C13 203.1 mm to (-16.2, 26.2), turned to 90 degrees
- moved R10 203.0 mm to (-19.7, -10.5), turned to 90 degrees
- moved C7 202.5 mm to (-29.7, 2.42), turned to 90 degrees
- moved R4 201.5 mm to (20.7, 4.97), turned to 90 degrees
- moved R26 186.3 mm to (-3.29, -2.09)
- moved D2 185.7 mm to (-29.5, 10.1), turned to 90 degrees
- moved U3 170.7 mm to (-14.7, 75.6), turned to 90 degrees
- moved C2 162.0 mm to (-16.8, 18.8), turned to 90 degrees
- moved R7 160.9 mm to (-3.69, -12.6)
- moved P4 159.9 mm to (-28.5, 27.0), turned to 90 degrees
- moved J1 158.3 mm to (-25.3, 126.5), turned to 90 degrees
- moved C6 155.9 mm to (-5.13, 26.8), turned to 90 degrees
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Connections:
- 1N1 pad 1: VCC -> +5V
- 1N3 pad 1: VCC -> +5V
- C1 pad 1: Net-(C1-Pad1) -> /V_CTRL
- C12 pad 1: VCC -> +5V
- D1 pad 1: VCC -> +5V
- D2 pad 2: VCC -> +5V
- P13 pad 1: VCC -> +5V
- P17 pad 1: VCC -> /+24V(EXT)
- P17 pad 2: /SPINDLE_EN -> /LIG/DESL
- P18 pad 1: VCC -> +5V
- P26 pad 1: VCC -> /CW/STOP
- P26 pad 2: Net-(1N4-Pad2) -> /+24V(EXT)
- P27 pad 2: Net-(P27-Pad2) -> GND
- P8 pad 1: /V_CTRL -> Net-(P8-Pad1)
- Q2 pad 1: /SPINDLE_EN -> Net-(Q2-Pad1)
- Q4 pad 1: Net-(1N4-Pad2) -> Net-(Q4-Pad1)
- R1 pad 2: Net-(C1-Pad1) -> /V_CTRL
- R14 pad 2: /V_REF -> Net-(R14-Pad2)
- R15 pad 1: VCC -> Net-(Q2-Pad1)
- R15 pad 2: Net-(Q2-Pad2) -> /SPINDLE_EN
- R16 pad 1: VCC -> +5V
- R27 pad 1: Net-(Q5-Pad2) -> /SPINDLE_EN
- R27 pad 2: /SPINDLE_EN -> Net-(Q5-Pad2)
- R28 pad 1: Net-(Q4-Pad2) -> /+24V(EXT)
- R28 pad 2: /SPINDLE_DIR -> /LIG/DESL
- R29 pad 1: Net-(P27-Pad2) -> Net-(Q4-Pad2)
- R29 pad 2: Net-(Q5-Pad2) -> /SPINDLE_DIR
- R3 pad 2: /V_CTRL -> Net-(P8-Pad1)
- R30 pad 2: VCC -> +5V
- R31 pad 1: VCC -> +5V
- R5 pad 2: /V_REF -> /SPINDLE_EN
- R6 pad 1: VCC -> Net-(Q2-Pad1)
- R6 pad 2: Net-(Q1-Pad2) -> +5V
- R7 pad 1: VCC -> +5V
- U1 pad 3: Net-(C1-Pad1) -> /V_CTRL
- U1 pad 6: /V_CTRL -> Net-(P8-Pad1)
- U1 pad 7: VCC -> +5V
- U2 pad 2: /V_REF -> Net-(R14-Pad2)
- U2 pad 6: /V_REF -> Net-(R14-Pad2)
- U2 pad 7: VCC -> +5V
- U3 pad 1: (no net) -> /SPINDLE_EN
- U3 pad 2: (no net) -> GND
- U3 pad 4: /Z_LIMIT_B -> /GND(EXT)
- U3 pad 5: /Z_LIMIT_A -> /LIG/DESL
- U3 pad 6: /Z_LIMIT* -> Net-(U3-Pad6)
- U4 pad 1: VCC -> +5V
Routing:
- net (no net): track 0.00 -> 3861.1 mm
- net GND: track 713.5 -> 0.00 mm, vias 17 -> 0
- net +5V: track 310.5 -> 0.00 mm, vias 10 -> 0
- net VCC: track 294.2 -> 0.00 mm, vias 10 -> 0
- net /X_STEP: track 262.7 -> 0.00 mm
- net /Y_STEP: track 228.4 -> 0.00 mm
- net /Z_STEP: track 195.2 -> 0.00 mm
- net /STEPPER_EN: track 182.6 -> 0.00 mm, vias 5 -> 0
- net /Z_DIR: track 129.0 -> 0.00 mm, vias 2 -> 0
- net /Y_DIR: track 127.5 -> 0.00 mm, vias 2 -> 0
- net /X_DIR: track 122.2 -> 0.00 mm, vias 2 -> 0
- net /X_LIMIT_B: track 114.3 -> 0.00 mm
- net /PROBE*: track 114.0 -> 0.00 mm
- net /START/RESUME*: track 109.3 -> 0.00 mm
- net /Z_LIMIT_B: track 105.3 -> 0.00 mm
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- removed copper zone on F.Cu, net GND
Other:
- board outline removed
- net class Default: trace_width 0.8 -> 1
