File: JB_CNC.kicad_pcb (KiCad board)
At the start: 2 copper layers, 100 x 150 mm, 90 parts, among them CON1 POWER_IN, J1 Arduino_Header, P1 Z_CTRL, P10 X_LIMIT_1, P11 Y_LIMIT_1, P12 Z_LIMIT_1, P13 FLUIDO, P14 X_LIMIT_2, P15 Y_LIMIT_2, P16 Z_LIMIT_2, P17 SPINDLE_PWR, P18 SPINDLE_LED, P19 SPINDLE_DIRECTION, P2 Z_LIMIT, P20 RESET/ABORT, P21 START/RESUME, P210 earth, P211 earth, P22 FEED_HOLD, P23 SAFETY_DOOR, P24 ASPIRADOR, P25 earth, P26 earth, P27 earth, P28 earth, P29 earth, P3 Y_CTRL, P4 Y_LIMIT, P5 X_CTRL, P6 X_LIMIT, P7 USB_TO_ARDUINO, P8 F_INV, P9 USB_SHIELD_INPUT, Q1 BC546, Q2 BC546, Q3 BC546, Q4 BC546, Q5 BC817-40, U1 CA3140, U2 LM7805CT, U3 CA3140, U4 74LS86, U6 LM7815ACT, u657 1N4001

Commit message: Circuito Redesenhado
Parts:
- removed 1N2, DFDSF1, u657: 1N4001, Diodes_ThroughHole:Diode_DO-35_SOD27_Horizontal_RM10
- removed C17, C18, C19: 4u7, Capacitors_ThroughHole:C_Radial_D5_L11_P2.5
- removed CON1: POWER_IN, Connect:BARREL_JACK
- removed G***: LOGO, triangulos_cta:15ffab
- removed G***: LOGO, triangulos_cta:15fcu
- removed P210, P211, P28, P29: earth, Socket_Strips:Socket_Strip_Straight_1x01
- added 1N3: 1N4001, Diodes_ThroughHole:Diode_DO-35_SOD27_Horizontal_RM10, F.Cu at (51.5, 134.3)
- added C10: 1uF, Capacitors_ThroughHole:C_Radial_D5_L11_P2.5, F.Cu at (12.9, 50.5)
- added C4: 1uF, Capacitors_ThroughHole:C_Radial_D5_L11_P2.5, F.Cu at (-29.7, -4.43)
- added C8: 1uF, Capacitors_ThroughHole:C_Radial_D5_L11_P2.5, F.Cu at (9.51, 39.2)
- added C9: 1uF, Capacitors_ThroughHole:C_Radial_D5_L11_P2.5, F.Cu at (41.3, 77.5)
- added D3: 1K5E68A, Diodes_ThroughHole:Diode_P600_Vertical_KathodeUp, F.Cu at (-26.5, 54.7)
- added R28: 4k7, Resistors_ThroughHole:Resistor_Vertical_RM5mm, F.Cu at (46.8, 49.8)
- added R29: 10k, Resistors_ThroughHole:Resistor_Vertical_RM5mm, F.Cu at (-11.7, -12.6)
- added R30: 4k7, Resistors_ThroughHole:Resistor_Vertical_RM5mm, F.Cu at (28.8, 26.0)
- added R31: 1k, Resistors_ThroughHole:Resistor_Vertical_RM5mm, F.Cu at (20.8, 15.5)
- added R32: 4k7, Resistors_ThroughHole:Resistor_Vertical_RM5mm, F.Cu at (54.8, 51.8)
- added R33: 1k, Resistors_ThroughHole:Resistor_Vertical_RM5mm, F.Cu at (43.5, 38.3)
- added R34: 1k, Resistors_ThroughHole:Resistor_Vertical_RM5mm, F.Cu at (12.9, 26.0)
- added R35: 4k7, Resistors_ThroughHole:Resistor_Vertical_RM5mm, F.Cu at (-11.3, -2.09)
- added R36: 1k, Resistors_ThroughHole:Resistor_Vertical_RM5mm, F.Cu at (4.70, -2.09)
- added R37: 4k7, Resistors_ThroughHole:Resistor_Vertical_RM5mm, F.Cu at (53.8, 62.3)
- added U10: 74LS32, Housings_DIP:DIP-14_W7.62mm_LongPads, F.Cu at (13.6, 145.4)
- added U5: 4N25, Housings_DIP:DIP-6_W7.62mm_LongPads, F.Cu at (30.0, 112.3)
- added W1: FONTE, Connect:bornier2, F.Cu at (44.8, 106.7)
- C1: value u47 -> 1uF
- C11, C5, C6, C7: value 4u7 -> 1uF
- C12: value 4u7 -> 100u; footprint Capacitors_ThroughHole:C_Radial_D5_L11_P2.5 -> Capacitors_ThroughHole:C_Radial_D10_L13_P5
- C13: value 4u7 -> 10u; footprint Capacitors_ThroughHole:C_Radial_D5_L11_P2.5 -> Capacitors_ThroughHole:C_Radial_D6.3_L11.2_P2.5
- C2: value 100u -> 1uF
- C3: value 10u -> 1uF
- D1: footprint Diodes_ThroughHole:Diode_P600_Vertical_AnodeUp -> Diodes_ThroughHole:Diode_P600_Vertical_KathodeUp
- D2: value LED -> LED_PWR
- J1: value Arduino_Header -> Arduino_Nano_Header; footprint cta_arduinos:arduino_uno_header -> w_conn_misc:arduino_nano_header
- P13: value FLUIDO -> ASPIRADOR
- P17: footprint w_conn_kk100:kk100_22-23-2021 -> w_conn_kk100:kk100_22-23-2031
- P18: value SPINDLE_LED -> FLUIDO
- P19: value SPINDLE_DIRECTION -> RESETA/INTERROMPE
- P20: value RESET/ABORT -> INICIA/CONTINUA
- P21: value START/RESUME -> PAUSA
- P22: value FEED_HOLD -> SONDA
- P23: value SAFETY_DOOR -> PORTA_SEGURANÇA
- P24: value ASPIRADOR -> earth; footprint w_conn_kk100:kk100_22-23-2021 -> w_details:hole_1mm
- P25: value earth -> SPINDLE_LED_ON; footprint Socket_Strips:Socket_Strip_Straight_1x01 -> w_conn_kk100:kk100_22-23-2021
- P26: value earth -> DIREÇÃO; footprint Socket_Strips:Socket_Strip_Straight_1x01 -> w_conn_kk100:kk100_22-23-2041
- P27: value earth -> SPINDLE_LED_OFF; footprint Socket_Strips:Socket_Strip_Straight_1x01 -> w_conn_kk100:kk100_22-23-2021
- P7: value USB_TO_ARDUINO -> USB_PARA_ARDUINO; footprint Connect:USB_A -> w_conn_pc:conn_usb_A
- P9: value USB_SHIELD_INPUT -> ENTRADA_USB_SHIELD; footprint Connect:USB_B -> w_conn_pc:conn_usb_B
- Q5: value BC817-40 -> BC546
- R1: value 100k -> 10k; footprint Resistors_ThroughHole:Resistor_Horizontal_RM10mm -> Resistors_ThroughHole:Resistor_Vertical_RM5mm
- R10, R11, R12, R21, R23, R8, R9: value 22k -> 10k
- R13, R27: value 1k -> 10k; footprint Resistors_ThroughHole:Resistor_Horizontal_RM10mm -> Resistors_ThroughHole:Resistor_Vertical_RM5mm
- R14: value 2k2 -> 10k; footprint Resistors_ThroughHole:Resistor_Horizontal_RM10mm -> Resistors_ThroughHole:Resistor_Vertical_RM5mm
- R15: value 10k -> 470; footprint Resistors_ThroughHole:Resistor_Horizontal_RM10mm -> Resistors_ThroughHole:Resistor_Vertical_RM5mm
- R16: value 100 -> 68k; footprint Resistors_ThroughHole:Resistor_Horizontal_RM10mm -> Resistors_ThroughHole:Resistor_Vertical_RM5mm
- R17, R25, R4, R5: footprint Resistors_ThroughHole:Resistor_Horizontal_RM10mm -> Resistors_ThroughHole:Resistor_Vertical_RM5mm
- R18, R6: value 100 -> 1k; footprint Resistors_ThroughHole:Resistor_Horizontal_RM10mm -> Resistors_ThroughHole:Resistor_Vertical_RM5mm
- R19: value 2k7 -> 1k; footprint Resistors_ThroughHole:Resistor_Horizontal_RM10mm -> Resistors_ThroughHole:Resistor_Vertical_RM5mm
- R2: value 10k -> 20k; footprint Resistors_ThroughHole:Resistor_Horizontal_RM10mm -> Resistors_ThroughHole:Resistor_Vertical_RM5mm
- R20: value 100 -> 10k; footprint Resistors_ThroughHole:Resistor_Horizontal_RM10mm -> Resistors_ThroughHole:Resistor_Vertical_RM5mm
- R22: value 22k -> 1k
- R24: value 2k2 -> 1k; footprint Resistors_ThroughHole:Resistor_Horizontal_RM10mm -> Resistors_ThroughHole:Resistor_Vertical_RM5mm
- R26: value 1k -> 2k2; footprint Resistors_ThroughHole:Resistor_Horizontal_RM10mm -> Resistors_ThroughHole:Resistor_Vertical_RM5mm
- R3: value 10k -> 22k; footprint Resistors_ThroughHole:Resistor_Horizontal_RM10mm -> Resistors_ThroughHole:Resistor_Vertical_RM5mm
- R7: value 22k -> 68k
- U2: value LM7805CT -> CA3140; footprint Power_Integrations:TO-220 -> Housings_DIP:DIP-8_W7.62mm_LongPads
- U3: value CA3140 -> 4N25; footprint Housings_DIP:DIP-8_W7.62mm_LongPads -> Housings_DIP:DIP-6_W7.62mm_LongPads
- U4: value 74LS86 -> LM7805CT; footprint Housings_DIP:DIP-14_W7.62mm_LongPads -> Power_Integrations:TO-220
- U6: value LM7815ACT -> 4N25; footprint Power_Integrations:TO-220 -> Housings_DIP:DIP-6_W7.62mm_LongPads
- moved R22 183.6 mm to (-0.78, 8.41), turned to 90 degrees
- moved D2 173.9 mm to (-29.5, 10.1), turned to 90 degrees
- moved R4 167.9 mm to (20.7, 4.97), turned to 90 degrees
- moved C2 165.4 mm to (-16.8, 18.8), turned to 90 degrees
- moved P6 163.1 mm to (-28.5, 17.4), turned to 90 degrees
- moved R10 160.8 mm to (-19.7, -10.5), turned to 90 degrees
- moved R7 155.2 mm to (-3.69, -12.6), turned to 90 degrees
- moved C11 154.3 mm to (-18.8, 10.4), turned to 90 degrees
- moved P21 152.4 mm to (-0.12, 77.8)
- moved P10 152.2 mm to (-15.0, 35.1), turned to 90 degrees
- moved P3 151.9 mm to (-11.7, 47.9)
- moved P4 144.3 mm to (-28.5, 27.0), turned to 90 degrees
- moved R19 144.0 mm to (19.5, 36.5), turned to 90 degrees
- moved C5 144.0 mm to (-6.33, 18.8), turned to 90 degrees
- moved R24 143.9 mm to (20.8, 26.0), turned to 90 degrees
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Connections:
- net /COOLANT_OUT renamed Net-(1N1-Pad2)
- 1N1 pad 1: +15V -> +5V
- C1 pad 1: Net-(C1-Pad1) -> /V_CTRL
- C11 pad 1: /X_LIMIT_2 -> /FEED_HOLD*
- C12 pad 1: /Y_LIMIT_2 -> +5V
- C13 pad 1: /Z_LIMIT_2 -> +5V
- C2 pad 1: +15V -> /X_LIMIT_A
- C3 pad 1: +5V -> /Y_LIMIT_A
- C5 pad 1: /X_LIMIT_1 -> /X_LIMIT_B
- C6 pad 1: /Y_LIMIT_1 -> /Y_LIMIT_B
- C7 pad 1: /Z_LIMIT_1 -> /Z_LIMIT_B
- D1 pad 1: Net-(D1-Pad1) -> +5V
- D2 pad 2: +15V -> +5V
- J1 pad 1: (no net) -> Net-(J1-Pad1)
- J1 pad 10: /FEED_HOLD -> /Z_DIR
- J1 pad 11: /START/RESUME -> /STEPPER_EN
- J1 pad 12: /COOLANT_EN -> /X_LIMIT*
- J1 pad 13: Net-(J1-Pad13) -> /Y_LIMIT*
- J1 pad 14: /PROBE -> /SPINDLE_PWM
- J1 pad 15: Net-(J1-Pad15) -> /Z_LIMIT*
- J1 pad 16: Net-(J1-Pad16) -> /SPINDLE_DIR
- J1 pad 17: /X_STEP -> Net-(J1-Pad17)
- J1 pad 18: /Y_STEP -> Net-(J1-Pad18)
- J1 pad 19: /Z_STEP -> /RESET/ABORT*
- J1 pad 20: /X_DIR -> /FEED_HOLD*
- J1 pad 21: /Y_DIR -> /START/RESUME*
- J1 pad 22: /Z_DIR -> /COOLANT_EN
- J1 pad 23: /STEPPER_EN -> Net-(J1-Pad23)
- J1 pad 24: /X_LIMIT -> /PROBE*
- J1 pad 25: /Y_LIMIT -> Net-(J1-Pad25)
- J1 pad 26: /SPINDLE_PWM -> Net-(J1-Pad26)
- J1 pad 27: /Z_LIMIT -> +5V
- J1 pad 28: /SPINDLE_DIR -> GND
- J1 pad 3: Net-(J1-Pad3) -> GND
- J1 pad 30: Net-(J1-Pad30) -> +5V
- J1 pad 4: Net-(J1-Pad4) -> GND
- J1 pad 5: Net-(J1-Pad5) -> /X_STEP
- J1 pad 6: GND -> /Y_STEP
- J1 pad 7: GND -> /Z_STEP
- J1 pad 8: +5V -> /X_DIR
- J1 pad 9: /RESET/ABORT -> /Y_DIR
- P10 pad 3: /X_LIMIT_1 -> Net-(P10-Pad3)
- P11 pad 3: /Y_LIMIT_1 -> Net-(P11-Pad3)
- P12 pad 3: /Z_LIMIT_1 -> Net-(P12-Pad3)
- P13 pad 1: Net-(P13-Pad1) -> +5V
- P14 pad 3: /X_LIMIT_2 -> Net-(P14-Pad3)
- P15 pad 3: /Y_LIMIT_2 -> Net-(P15-Pad3)
- P16 pad 3: /Z_LIMIT_2 -> Net-(P16-Pad3)
- P17 pad 1: Net-(P17-Pad1) -> /+24V(EXT)
- P17 pad 2: /SPINDLE_EN -> /LIG/DESL
- P18 pad 1: Net-(P18-Pad1) -> +5V
- P18 pad 2: GND -> Net-(1N3-Pad2)
- P19 pad 1: Net-(P19-Pad1) -> +5V
- P19 pad 2: /SPINDLE_EN -> Net-(P19-Pad2)
- P2 pad 1: /Z_LIMIT_1 -> /Z_LIMIT_A
- P2 pad 2: /Z_LIMIT_2 -> /Z_LIMIT_B
- P20 pad 2: /RESET/ABORT -> Net-(P20-Pad2)
- P21 pad 2: /START/RESUME -> /SAFETY_IN
- P22 pad 1: +5V -> GND
- P22 pad 2: /SAFETY_IN -> Net-(P22-Pad2)
- P23 pad 3: /FEED_HOLD -> Net-(P23-Pad3)
- P24 pad 1: Net-(P24-Pad1) -> GND
- P25 pad 1: Earth -> Net-(P25-Pad1)
- P26 pad 1: Earth -> /CW/STOP
- P27 pad 1: Earth -> Net-(P27-Pad1)
- P4 pad 1: /Y_LIMIT_1 -> /Y_LIMIT_A
- P4 pad 2: /Y_LIMIT_2 -> /Y_LIMIT_B
- P6 pad 1: /X_LIMIT_1 -> /X_LIMIT_A
- P6 pad 2: /X_LIMIT_2 -> /X_LIMIT_B
- P7 pad 5: Earth -> GND
- P8 pad 1: /V_CTRL -> Net-(P8-Pad1)
- P9 pad 5: Earth -> GND
- Q2 pad 1: /SPINDLE_EN -> Net-(Q2-Pad1)
- Q3 pad 1: /SPINDLE_EN -> Net-(1N3-Pad2)
- Q4 pad 1: /PROBE_OUT -> Net-(Q4-Pad1)
- Q5 pad 1: Net-(Q5-Pad1) -> Net-(P25-Pad2)
- Q5 pad 2: GND -> Net-(Q5-Pad2)
- Q5 pad 3: /SPINDLE_OUT -> GND
- R1 pad 2: Net-(C1-Pad1) -> /V_CTRL
- R10 pad 1: /X_LIMIT_2 -> Net-(P12-Pad3)
- R10 pad 2: GND -> /Z_LIMIT_A
- R11 pad 1: /Y_LIMIT_2 -> Net-(P14-Pad3)
- R11 pad 2: GND -> /X_LIMIT_B
- R12 pad 1: /Z_LIMIT_2 -> Net-(P15-Pad3)
- R12 pad 2: GND -> /Y_LIMIT_B
- R13 pad 1: GND -> Net-(P16-Pad3)
- R13 pad 2: Net-(R13-Pad2) -> /Z_LIMIT_B
- R14 pad 1: Net-(R13-Pad2) -> Net-(Q2-Pad2)
- R15 pad 1: Net-(Q2-Pad2) -> Net-(Q2-Pad1)
- R15 pad 2: Net-(R14-Pad2) -> /SPINDLE_EN
- R16 pad 1: +15V -> +5V
- R16 pad 2: Net-(P17-Pad1) -> Net-(Q2-Pad2)
- R17 pad 2: /SPINDLE_DIR -> /COOLANT_EN
- R18 pad 1: +15V -> GND
- R18 pad 2: Net-(P19-Pad1) -> Net-(P19-Pad2)
- R19 pad 1: Net-(Q4-Pad2) -> GND
- R19 pad 2: /PROBE -> Net-(P20-Pad2)
- R20 pad 1: +15V -> /RESET/ABORT*
- R20 pad 2: Net-(P24-Pad1) -> Net-(P19-Pad2)
- R21 pad 1: /RESET/ABORT -> /START/RESUME*
- R21 pad 2: GND -> Net-(P20-Pad2)
- R22 pad 1: /START/RESUME -> Net-(P22-Pad2)
- R23 pad 1: /FEED_HOLD -> /PROBE*
- R23 pad 2: GND -> Net-(P22-Pad2)
- R24 pad 1: Net-(D2-Pad1) -> GND
- R24 pad 2: GND -> /SAFETY_IN
- R25 pad 1: Net-(Q5-Pad1) -> /FEED_HOLD*
- R25 pad 2: /SPINDLE_EN -> Net-(P23-Pad3)
- R26 pad 1: +15V -> Net-(D2-Pad1)
- R26 pad 2: /SPINDLE_OUT -> GND
- R27 pad 1: Net-(P18-Pad1) -> /SPINDLE_EN
- R27 pad 2: /SPINDLE_OUT -> Net-(Q5-Pad2)
- R3 pad 1: /V_CTRL -> Net-(R2-Pad2)
- R3 pad 2: Net-(R2-Pad2) -> Net-(P8-Pad1)
- R5 pad 2: /COOLANT_EN -> /SPINDLE_EN
- R6 pad 1: +15V -> Net-(Q2-Pad1)
- R6 pad 2: Net-(P13-Pad1) -> +5V
- R7 pad 1: /X_LIMIT_1 -> +5V
- R7 pad 2: GND -> Net-(Q1-Pad2)
- R8 pad 1: /Y_LIMIT_1 -> Net-(P10-Pad3)
- R8 pad 2: GND -> /X_LIMIT_A
- R9 pad 1: /Z_LIMIT_1 -> Net-(P11-Pad3)
- R9 pad 2: GND -> /Y_LIMIT_A
- U1 pad 3: Net-(C1-Pad1) -> /V_CTRL
- U1 pad 6: /V_CTRL -> Net-(P8-Pad1)
- U1 pad 7: +15V -> +5V
- U2 pad 1: +15V -> Net-(U2-Pad1)
- U2 pad 2: GND -> Net-(R14-Pad2)
- U2 pad 3: +5V -> /V_CTRL
- U3 pad 1: Net-(U3-Pad1) -> /SPINDLE_EN
- U3 pad 2: Net-(R13-Pad2) -> GND
- U3 pad 3: /V_CTRL -> (no net)
- U3 pad 4: GND -> /GND(EXT)
- U3 pad 5: Net-(U3-Pad5) -> /LIG/DESL
- U3 pad 6: Net-(R14-Pad2) -> Net-(U3-Pad6)
- U4 pad 1: /X_LIMIT_1 -> +5V
- U4 pad 2: /X_LIMIT_2 -> GND
- U4 pad 3: /X_LIMIT -> +5V
- U6 pad 1: Net-(D1-Pad1) -> Net-(R34-Pad1)
- U6 pad 3: +15V -> (no net)
Routing:
- net (no net): track 0.00 -> 3861.1 mm
- net GND: track 762.4 -> 0.00 mm, vias 14 -> 0
- net +5V: track 406.8 -> 0.00 mm, vias 5 -> 0
- net +15V: track 281.3 -> 0.00 mm, vias 2 -> 0
- net /SPINDLE_EN: track 113.5 -> 0.00 mm
- net /STEPPER_EN: track 89.2 -> 0.00 mm
- net /SPINDLE_DIR: track 76.1 -> 0.00 mm
- net /Z_LIMIT: track 73.1 -> 0.00 mm
- net /X_LIMIT_1: track 57.3 -> 0.00 mm
- net /X_LIMIT_2: track 56.7 -> 0.00 mm
- net /X_DIR: track 54.3 -> 0.00 mm, vias 2 -> 0
- net /Z_DIR: track 53.2 -> 0.00 mm
- net Net-(P7-Pad2): track 52.9 -> 0.00 mm
- net /Y_DIR: track 52.5 -> 0.00 mm, vias 2 -> 0
- net /RESET/ABORT: track 50.4 -> 0.00 mm
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- removed copper zone on F.Cu, net Earth
Other:
- board outline removed
- net class Alimentação added: clearance 0.6, trace_width 1.4, via_dia 1.6, via_drill 0.8
- net class Default: trace_width 0.8 -> 1
- net class Potencia removed
- rule pad_to_mask_clearance: 0.2 -> 0
- board text removed: "Controle CPVR 02"

Commit message: Desenho parcial da placa
Parts:
- added F1: Fuse, w_misc_comp:fuse_holder_CQ-2, F.Cu at (173.1, 252.4)
- R1, R10, R11, R12, R13, R14, R15, R16, R17, R18, R19, R2, R20, R21, R22, R23, R24, R25, R26, R27, R28, R29, R3, R30, R31, R32, R33, R34, R35, R36, R37, R4, R5, R6, R7, R8, R9: footprint Resistors_ThroughHole:Resistor_Vertical_RM5mm -> w_pth_resistors:rc07_vert
- moved R29 425.7 mm to (279.9, 297.5), turned to 0 degrees
- moved R7 420.0 mm to (288.0, 289.6), turned to 0 degrees
- moved R3 419.6 mm to (324.8, 258.3), turned to 0 degrees
- moved R1 415.5 mm to (309.0, 286.2), turned to 0 degrees
- moved R26 410.7 mm to (314.3, 258.3), turned to 0 degrees
- moved Q2 407.4 mm to (327.0, 267.0), turned to 0 degrees
- moved R35 407.2 mm to (290.7, 271.1), turned to 0 degrees
- moved R17 406.8 mm to (269.7, 286.4), turned to 0 degrees
- moved D2 400.0 mm to (309.3, 222.7), turned to 0 degrees
- moved R4 397.4 mm to (298.0, 289.6), turned to 0 degrees
- moved C11 397.1 mm to (316.9, 222.6), turned to 0 degrees
- moved R36 396.5 mm to (318.9, 239.8), turned to 0 degrees
- moved Q1 392.8 mm to (285.2, 306.2), turned to 0 degrees
- moved R15 391.9 mm to (298.0, 252.3), turned to 0 degrees
- moved R27 388.7 mm to (298.5, 279.1), turned to 0 degrees
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Connections:
- 1N1 pad 1: +5V -> +14.2V
- 1N3 pad 1: +5V -> +14.2V
- C12 pad 1: +5V -> +14.2V
- D1 pad 1: +5V -> +14.2V
- D2 pad 2: +5V -> +14.2V
- D3 pad 1: +5V -> +14.2V
- J1 pad 17: Net-(J1-Pad17) -> (no net)
- J1 pad 23: Net-(J1-Pad23) -> (no net)
- J1 pad 25: Net-(J1-Pad25) -> (no net)
- J1 pad 26: Net-(J1-Pad26) -> (no net)
- P13 pad 1: +5V -> +14.2V
- P18 pad 1: +5V -> +14.2V
- P2 pad 1: /Z_LIMIT_A -> GND
- P2 pad 3: GND -> /Z_LIMIT_A
- P4 pad 1: /Y_LIMIT_A -> GND
- P4 pad 3: GND -> /Y_LIMIT_A
- P6 pad 1: /X_LIMIT_A -> GND
- P6 pad 3: GND -> /X_LIMIT_A
- R7 pad 1: +5V -> +14.2V
- U1 pad 7: +5V -> +14.2V
- U10 pad 1: /X_LIMIT_A -> /Y_LIMIT_B
- U10 pad 10: /Z_LIMIT_B -> (no net)
- U10 pad 11: (no net) -> /Z_LIMIT*
- U10 pad 12: (no net) -> /Z_LIMIT_B
- U10 pad 13: (no net) -> /Z_LIMIT_A
- U10 pad 2: /X_LIMIT_B -> /Y_LIMIT_A
- U10 pad 3: /X_LIMIT* -> /Y_LIMIT*
- U10 pad 4: /Y_LIMIT_A -> /X_LIMIT_B
- U10 pad 5: /Y_LIMIT_B -> /X_LIMIT_A
- U10 pad 6: /Y_LIMIT* -> /X_LIMIT*
- U10 pad 8: /Z_LIMIT* -> (no net)
- U10 pad 9: /Z_LIMIT_A -> (no net)
- U2 pad 7: +5V -> +14.2V
- U4 pad 1: +5V -> +14.2V
- W1 pad 2: Net-(D1-Pad2) -> Net-(F1-Pad2)
Routing:
- net (no net): track 3861.1 -> 0.00 mm
- net GND: track 0.00 -> 442.5 mm, vias 0 -> 6
- net /STEPPER_EN: track 0.00 -> 202.3 mm, vias 0 -> 6
- net +5V: track 0.00 -> 175.6 mm, vias 0 -> 5
- net /Z_STEP: track 0.00 -> 168.4 mm
- net /Z_DIR: track 0.00 -> 145.1 mm, vias 0 -> 2
- net /Y_STEP: track 0.00 -> 141.5 mm
- net /Y_DIR: track 0.00 -> 127.1 mm, vias 0 -> 2
- net /X_STEP: track 0.00 -> 114.6 mm
- net /X_DIR: track 0.00 -> 110.2 mm, vias 0 -> 2
- net /Z_LIMIT*: track 0.00 -> 69.2 mm
- net /Y_LIMIT*: track 0.00 -> 64.2 mm
- net /X_LIMIT*: track 0.00 -> 50.7 mm
- net /X_LIMIT_A: track 0.00 -> 48.7 mm
- net /X_LIMIT_B: track 0.00 -> 45.1 mm
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Other:
- board outline added: 90 x 192 mm
- net class Default: trace_width 1 -> 0.9
