File: JB_CNC.sch (KiCad schematic (older format))
At the start: 89 parts, among them J1 Arduino_Nano_Header, P1 Z_CTRL, P10 X_LIMIT_1, P11 Y_LIMIT_1, P12 Z_LIMIT_1, P13 ASPIRADOR, P14 X_LIMIT_2, P15 Y_LIMIT_2, P16 Z_LIMIT_2, P17 SPINDLE_PWR, P18 FLUIDO, P19 RESETA/INTERROMPE, P2 Z_LIMIT, P20 INICIA/CONTINUA, P21 PAUSA, P22 SONDA, P23 PORTA_SEGURANÇA, P24 earth, P25 SPINDLE_LED_ON, P26 DIREÇÃO_SPINDLE, P27 SPINDLE_LED_OFF, P3 Y_CTRL, P4 Y_LIMIT, P5 X_CTRL, P6 X_LIMIT, P7 USB_PARA_ARDUINO, P8 F_INV, P9 ENTRADA_USB_SHIELD, Q1 BC546, Q2 BC546, Q3 BC546, Q4 BC546, Q5 BC546, U1 CA3140, U10 74LS32, U2 CA3140, U4 LM7805CT

Commit message: Modificado módulo SPINDLE
Parts:
- removed 1N2, 1N4: 1N4001, Diodes_ThroughHole:Diode_DO-35_SOD27_Horizontal_RM10, symbol D
- removed P17: SPINDLE_PWR, w_conn_kk100:kk100_22-23-2021, symbol CONN_01X02
- removed P26: DIREÇÃO_SPINDLE, w_conn_kk100:kk100_22-23-2021, symbol CONN_01X02
- removed Q4: BC546, TO_SOT_Packages_THT:TO-92_Inline_Wide, symbol BC546
- removed R15: 680k, Resistors_ThroughHole:Resistor_Vertical_RM5mm, symbol R
- removed R28: 2k7, Resistors_ThroughHole:Resistor_Vertical_RM5mm, symbol R
- added P?: SPINDLE_PWR, symbol CONN_01X03
- added P?: SPINDLE_DIRECT, symbol CONN_01X03
- added Q?: BC546, TO_SOT_Packages_THT:TO-92_Inline_Wide, symbol BC546
- added R? (x2): 4k7, Resistors_ThroughHole:Resistor_Vertical_RM5mm, symbol R-RESCUE-JB_CNC
- added R? (x2): 470, Resistors_ThroughHole:Resistor_Vertical_RM5mm, symbol R-RESCUE-JB_CNC
- added R? (x2): 1k, Resistors_ThroughHole:Resistor_Vertical_RM5mm, symbol R-RESCUE-JB_CNC
- added R?: 10k, Resistors_ThroughHole:Resistor_Vertical_RM5mm, symbol R-RESCUE-JB_CNC
- added U? (x2): 4N25, DIP-6, symbol 4N25
- D2: symbol LED -> LED-RESCUE-JB_CNC
- R1, R10, R11, R12, R13, R16, R17, R18, R19, R2, R20, R21, R22, R23, R24, R25, R26, R27, R29, R3, R30, R31, R32, R4, R5, R6, R7, R8, R9: symbol R -> R-RESCUE-JB_CNC
- R14: value 2k7 -> 10k; symbol R -> R-RESCUE-JB_CNC
Connections:
- net labels added: +24V(EXT), GND(EXT), LIG/DESL
- wire segments 225 -> 250
- no-connect marks 13 -> 15
Other:
- moved on the sheet: U1

Commit message: Refeitos circuitos de acionamento do SPINDLE, ASPIRADOR e BOMBA
Parts:
- removed R27: 8k2, Resistors_ThroughHole:Resistor_Vertical_RM5mm, symbol R-RESCUE-JB_CNC
- removed R29: 1k, Resistors_ThroughHole:Resistor_Vertical_RM5mm, symbol R-RESCUE-JB_CNC
- removed R6: 680k, Resistors_ThroughHole:Resistor_Vertical_RM5mm, symbol R-RESCUE-JB_CNC
- added P?: CW/STOP, symbol CONN_01X03
- added R?: 1k, Resistors_ThroughHole:Resistor_Vertical_RM5mm, symbol R-RESCUE-JB_CNC
- added R?: 4k7, Resistors_ThroughHole:Resistor_Vertical_RM5mm, symbol R-RESCUE-JB_CNC
- added R?: 10k, Resistors_ThroughHole:Resistor_Vertical_RM5mm, symbol R-RESCUE-JB_CNC
- added U?: 4N25, DIP-6, symbol 4N25
- P?: value SPINDLE_DIRECT -> CCW/STOP
- R30, R32: value 10k -> 4k7
- R31: value 2k2 -> 1k
- R?: value 470 -> 1k
Connections:
- net labels added: CCW/STOP, CW/STOP
- net labels removed: V_REF
- wire segments 250 -> 252
- no-connect marks 15 -> 16
Other:
- note added: "Amplificação do sinal SPINDLE_DIR para utilização no \ninversor de frequência:\n\nO Inversor dispõe de duas entradas de controle de \ndireção: HORARIO/PARADO(CW/STOP) e \nANTIHORÁRIO/PARADO (CCW/STOP), que no caso de um\nestar ativado, o outro deve estar desativado.\nPara acionar um ou o outro, utiliza-se um circuito \ntransistorizado com optoisoladores para controlar esses\nsinais e isolar o cir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"
- note added: "Ativação do aspirador de acordo com spindle \n\nO aspirador deve sempre estar ligado enquanto\no spindle estiver em operação. Para isto, usa-se \num circuito transistorizado identico ao do spindle\nque ativa/desativa o relé do aspirador exatamente \nquando o relé de ativação do spindle for \nativado/desativado.\nDevido a altas correntes, foi colocado somente\no pino, pois o relé e o circuito de a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"
- note added: "Pino para e desativar o relé de alimentação\nda bomba de fluído arrefecedor.\n\nDevido a altas correntes, foi colocado somente\no pino, pois o relé e o circuito de alimentação \nda bomba serão colocados numa placa separada."
- note removed: "Amplificação do sinal SPINDLE_DIR para\nutilizar no inversor de frequência:\n\nO relé de ativação das entradas do inversor\nde frequência é do tipo 12V, portanto usa-se\num circuito transistorizado para amplificar o\nsinal do arduíno de 5 para VCC com corrente\nsuficiente para ativar o relé.\n"
- note removed: "Ativação do aspirador de acordo com spindle \n\nO aspirador deve sempre estar ligado enquanto\no spindle estiver em operação. Para isto, usa-se \num circuito transistorizado identico ao do spindle\nque ativa/desativa o relé do aspirador exatamente \nquando o relé de ativação do spindle for \nativado/desativado."
- note removed: "Pino para e desativar o relé de alimentação\nda bomba de fluído arrefecedor.\n\nDevido a altas correntes, foi colocado somente\no pino, pois o relé de alimentação da bomba \nserá colocado numa placa separada."

Commit message: Finalizado Esquema V0.2
Parts:
- removed P?: CCW/STOP, symbol CONN_01X03
- removed P?: CW/STOP, symbol CONN_01X03
- added D3: 1K5E68A, Diodes_ThroughHole:Diode_P600_Vertical_KathodeUp, symbol D_TVS
- added P26: DIREÇÃO, w_conn_kk100:kk100_22-23-2041, symbol CONN_01X04
- D2: footprint LEDs:LED-3MM -> LEDs:LED-5MM
- P17: renamed from P?; footprint (none) -> w_conn_kk100:kk100_22-23-2031
- R2: value 10k -> 20k
- R3: value 10k -> 22k
- U3, U5, U6: renamed from U?; footprint DIP-6 -> Housings_DIP:DIP-6_W7.62mm_LongPads
- gave numbers to parts that had none: 11
Other:
- note added: "Amplificação do sinal SPINDLE_DIR para utilização no \ninversor de frequência:\n\nO Inversor dispõe de duas entradas de controle de \ndireção: HORARIO/PARADO(CW/STOP) e \nANTIHORÁRIO/PARADO (CCW/STOP), que no caso de uma\nestar ativada (HIGH), a outra deve estar desativada.\nPara acionar uma ou a outra, utiliza-se um circuito \ntransistorizado com optoisoladores para controlar esses\nsinais e iso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"
- note added: "Fonte: 14.8 - 15VDC VCC: 14.1 - 14.4V\nDiodo Ultra Rápido para Polarização Reversa.\nDiodo TVS para surtos de tensão\nRegulador de Tensão para 5V.\n"
- note removed: "Amplificação do sinal SPINDLE_DIR para utilização no \ninversor de frequência:\n\nO Inversor dispõe de duas entradas de controle de \ndireção: HORARIO/PARADO(CW/STOP) e \nANTIHORÁRIO/PARADO (CCW/STOP), que no caso de um\nestar ativado, o outro deve estar desativado.\nPara acionar um ou o outro, utiliza-se um circuito \ntransistorizado com optoisoladores para controlar esses\nsinais e isolar o cir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"
- note removed: "Fonte: 14.8 - 15VDC VCC: 14.1 - 14.4V\nDiodo Ultra Rápido para Polarização Reversa.\nRegulador de Tensão para 5V."

Commit message: Desenho parcial da placa
Parts:
- added F1: Fuse, w_misc_comp:fuse_holder_CQ-2, symbol Fuse
Connections:
- net labels added: +14.2V
- net labels removed: VCC
- wire segments 252 -> 253
